File: diff_driver/diff_driver.sch (KiCad schematic (older format))
At the start: 16 parts, among them J1 CONN_01X07, J2 RJ45_LED, U1 am26ls31, U2 LDO

Commit message: parts
Parts:
- C1, C2, C3, C6: LCSC (none) -> C14663
- C4, C5, C7: LCSC (none) -> C15849
- R1, R2, R3: LCSC (none) -> C23018
- R4, R5: LCSC (none) -> C23204
- U1: LCSC (none) -> C6179
- U2: LCSC (none) -> C9055
Changed lines of the file:
@@
 F 2 "stmbl:C_0603" H 7088 1750 50  0001 C CNN
 F 3 "~" H 7050 1900 50  0001 C CNN
+F 4 "C14663" H 7050 1900 50  0001 C CNN "LCSC"
 	1    7050 1900
 	1    0    0    -1
@@
 F 2 "stmbl:C_0603" H 5188 5650 50  0001 C CNN
 F 3 "~" H 5150 5800 50  0001 C CNN
+F 4 "C14663" H 5150 5800 50  0001 C CNN "LCSC"
 	1    5150 5800
 	1    0    0    -1
@@
 F 2 "stmbl:R_0603" V 7980 3750 50  0001 C CNN
 F 3 "" H 8050 3750 50  0000 C CNN
+F 4 "C23204" H 8050 3750 50  0001 C CNN "LCSC"
 	1    8050 3750
 	0    1    1    0
@@
 F 2 "stmbl:R_0603" V 7980 4450 50  0001 C CNN
 F 3 "" H 8050 4450 50  0000 C CNN
+F 4 "C23204" H 8050 4450 50  0001 C CNN "LCSC"
 	1    8050 4450
 	0    1    1    0
@@
 F 2 "stmbl:R_0603" V 3480 3150 50  0001 C CNN
 F 3 "" H 3550 3150 50  0000 C CNN
+F 4 "C23018" H 3550 3150 50  0001 C CNN "LCSC"
 	1    3550 3150
 	0    1    1    0
@@
 F 2 "stmbl:R_0603" V 3480 3250 50  0001 C CNN
 F 3 "" H 3550 3250 50  0000 C CNN
+F 4 "C23018" H 3550 3250 50  0001 C CNN "LCSC"
 	1    3550 3250
 	0    1    1    0
@@
 F 2 "stmbl:R_0603" V 3480 3350 50  0001 C CNN
 F 3 "" H 3550 3350 50  0000 C CNN
+F 4 "C23018" H 3550 3350 50  0001 C CNN "LCSC"
 	1    3550 3350
 	0    1    1    0
@@
 F 2 "stmbl:SOIC-16" H 5050 3850 60  0001 C CNN
 F 3 "" H 5050 3850 60  0001 C CNN
+F 4 "C6179" H 5050 3850 50  0001 C CNN "LCSC"
 	1    5050 3850
 	1    0    0    -1
@@
 F 2 "stmbl:C_0603" H 5488 5650 50  0001 C CNN
 F 3 "~" H 5450 5800 50  0001 C CNN
+F 4 "C15849" H 5450 5800 50  0001 C CNN "LCSC"
 	1    5450 5800
 	1    0    0    -1
@@
 F 2 "stmbl:C_0603" H 6788 1750 50  0001 C CNN
 F 3 "~" H 6750 1900 50  0001 C CNN
+F 4 "C15849" H 6750 1900 50  0001 C CNN "LCSC"
 	1    6750 1900
 	1    0    0    -1
@@
 F 2 "stmbl:C_0603" H 6488 1750 50  0001 C CNN
 F 3 "~" H 6450 1900 50  0001 C CNN
+F 4 "C14663" H 6450 1900 50  0001 C CNN "LCSC"
 	1    6450 1900
 	1    0    0    -1
@@
 F 2 "stmbl:SOT-23-5" H 5750 1800 50  0001 C CIN
 F 3 "" H 5100 2050 50  0000 C CNN
+F 4 "C9055" H 5100 2050 50  0001 C CNN "LCSC"
 	1    5100 2050
 	1    0    0    -1
@@
 F 2 "stmbl:C_0603" H 5738 2000 50  0001 C CNN
 F 3 "~" H 5700 2150 50  0001 C CNN
+F 4 "C14663" H 5700 2150 50  0001 C CNN "LCSC"
 	1    5700 2150
 	0    1    1    0
@@
 F 2 "stmbl:C_0603" H 7388 1750 50  0001 C CNN
 F 3 "~" H 7350 1900 50  0001 C CNN
+F 4 "C15849" H 7350 1900 50  0001 C CNN "LCSC"
 	1    7350 1900
 	1    0    0    -1

Commit message: jlc export
Parts:
- removed C4, C7: 1u, stmbl:C_0603, symbol stmbl:C
- added C1, C2: 10u, stmbl:C_0805, symbol stmbl:C
- renumbered C2 to C101, C5 to C102, C6 to C103, C3 to C104, C1 to C106, J1 to J101, J2 to J102, R1 to R101, R2 to R102, R3 to R103, R4 to R104, R5 to R105, U1 to U101, U2 to U102
Connections:
- net +3V3: now also C1.1
- net +5V: now also C2.1
- net GND: now also C1.2, C2.2
