File: diff_driver/diff_driver.kicad_pcb (KiCad board)
At the start: 2 copper layers, 32 x 22 mm, 14 parts, among them J1 CONN_01X07, J2 RJ45_LED, U1 am26ls31, U2 HT75XX-1

Commit message: hw
Parts:
- added C6: 100n, stmbl:C_0603, F.Cu at (152.8, 82.5)
- added C7: 1u, stmbl:C_0603, F.Cu at (157.2, 85.0)
- C4, C5: value 1n -> 1u
- U2: value HT75XX-1 -> LDO; footprint stmbl:SOT-89-3 -> stmbl:SOT-23-5
- moved C1 4.07 mm to (156.0, 85.0)
- moved C3 2.14 mm to (150.5, 85.0)
- moved U2 1.54 mm to (153.2, 84.8), turned to 180 degrees
- moved C4 1.27 mm to (149.2, 85.0), turned to 90 degrees
- moved R4 0.10 mm to (159.0, 96.2)
Connections:
- U2 pad 1: GND -> +5V
- U2 pad 2: +5V -> GND
- U2 pad 3: +3V3 -> +5V
Routing:
- net +5V: track 24.2 -> 19.5 mm, vias 4 -> 5
- net Net-(J2-Pad5): track 19.6 -> 21.1 mm
- net +3V3: track 8.07 -> 6.62 mm
- net Net-(C6-Pad2): track 0.00 -> 1.32 mm
Other:
- net class Default: clearance 0.2 -> 0.15; trace_width 0.25 -> 0.2; via_dia 0.8 -> 0.6; via_drill 0.4 -> 0.3
- rule trace_clearance: 0.2 -> 0.15
- rule via_min_size: 0.4 -> 0.6

Commit message: hw
Other:
- board size 32 x 22 mm -> 30.5 x 22 mm
Changed lines of the file:
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@@
     (add_net "Net-(J2-Pad5)")
     (add_net "Net-(J2-Pad6)")
-    (add_net "Net-(U1-Pad13)")
-    (add_net "Net-(U1-Pad14)")
   )
   (module stmbl:C_0603 (layer F.Cu)
@@
     (effects (font (size 1.55 1.55) (thickness 0.25)) (justify right))
   )
-  (gr_text "8 GND\n7   5V\n5/4 Z\n3/6 B\n1/2 A" (at 168.75 91) (layer F.SilkS)
+  (gr_text "8 GND\n7 5V\n5/4 Z\n3/6 B\n1/2 A" (at 168.5 91) (layer F.SilkS)
     (effects (font (size 1 1) (thickness 0.2)) (justify left))
   )
@@
     (effects (font (size 1 1) (thickness 0.2)) (justify left mirror))
   )
-  (gr_arc (start 174 81) (end 175 81) (angle -90) (layer Edge.Cuts) (width 0.1))
-  (gr_arc (start 174 101) (end 174 102) (angle -90) (layer Edge.Cuts) (width 0.1))
+  (gr_arc (start 172.5 81) (end 173.5 81) (angle -90) (layer Edge.Cuts) (width 0.1))
+  (gr_arc (start 172.5 101) (end 172.5 102) (angle -90) (layer Edge.Cuts) (width 0.1))
   (gr_arc (start 144 101) (end 143 101) (angle -90) (layer Edge.Cuts) (width 0.1))
   (gr_arc (start 144 81) (end 144 80) (angle -90) (layer Edge.Cuts) (width 0.1))
@@
   )
   (gr_line (start 143 101) (end 143 81) (layer Edge.Cuts) (width 0.1))
-  (gr_line (start 174 102) (end 144 102) (layer Edge.Cuts) (width 0.1))
-  (gr_line (start 175 81) (end 175 101) (layer Edge.Cuts) (width 0.1))
-  (gr_line (start 144 80) (end 174 80) (layer Edge.Cuts) (width 0.1))
+  (gr_line (start 172.5 102) (end 144 102) (layer Edge.Cuts) (width 0.1))
+  (gr_line (start 173.5 81) (end 173.5 101) (layer Edge.Cuts) (width 0.1))
+  (gr_line (start 144 80) (end 172.5 80) (layer Edge.Cuts) (width 0.1))
   (segment (start 151.5 96.245) (end 151.55 96.195) (width 0.25) (layer F.Cu) (net 2))
   (segment (start 151.5 97.75) (end 151.5 96.245) (width 0.25) (layer F.Cu) (net 2))
@@
     (polygon
       (pts
-        (xy 144 81.5) (xy 144.5 81) (xy 173.5 81) (xy 174 81.5) (xy 174 100.5)
-        (xy 173.5 101) (xy 144.5 101) (xy 144 100.5)
+        (xy 144 81.5) (xy 144.5 81) (xy 172 81) (xy 172.5 81.5) (xy 172.5 100.5)
+        (xy 172 101) (xy 144.5 101) (xy 144 100.5)
       )
     )
@@
     (polygon
       (pts
-        (xy 144 81.5) (xy 144.5 81) (xy 173.5 81) (xy 174 81.499671) (xy 174 100.5)
-        (xy 173.5 101) (xy 144.49987 101) (xy 144 100.5)
+        (xy 144 81.5) (xy 144.5 81) (xy 172 81) (xy 172.5 81.499671) (xy 172.5 100.5)
+        (xy 172 101) (xy 144.49987 101) (xy 144 100.5)
       )
     )

Commit message: jlc export
Parts:
- removed C4, C7: 1u, stmbl:C_0603
- added C1: 10u, stmbl:C_0805, F.Cu at (149.5, 84.5)
- added C2: 10u, stmbl:C_0805, F.Cu at (158.0, 84.5)
- moved R105 2.50 mm to (159.0, 87.5)
- moved C103 0.50 mm to (153.2, 82.5)
- moved C104 0.50 mm to (151.0, 85.0)
- moved C106 0.50 mm to (156.5, 85.0)
- moved U102 0.50 mm to (153.8, 84.8)
- renumbered C2 to C101, C5 to C102, C6 to C103, C3 to C104, C1 to C106, J1 to J101, J2 to J102, R1 to R101, R2 to R102, R3 to R103, R4 to R104, R5 to R105, U1 to U101, U2 to U102
Routing:
- net Net-(J102-Pad5): track 21.1 -> 18.6 mm
- net Net-(J102-Pad10): track 1.97 -> 3.41 mm
- net +5V: track 19.5 -> 20.1 mm
