File: cmc/pcb.kicad_pcb (KiCad board)
At the start: 4 copper layers, 66.8 x 22 mm, 12 parts, among them J1 RJ45_LED, J2 RJ45_LED, U1 CMC, U11 CMC, U2 USBLC6-4SC6, U3 CMC, U4 CMC, U6 USBLC6-4SC6

Commit message: hw
Routing:
- net 13: track 45.2 -> 0.00 mm
- net +3V3: track 28.6 -> 39.2 mm, vias 2 -> 3
- added copper zone on B.Cu, net 13
Changed lines of the file:
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@@
     (thickness 1.6)
     (drawings 4)
-    (tracks 160)
+    (tracks 158)
     (zones 0)
     (modules 12)
@@
     (user_trace_width 1)
     (trace_clearance 0.15)
-    (zone_clearance 0.508)
+    (zone_clearance 0.2)
     (zone_45_only no)
     (trace_min 0.2)
@@
   (segment (start 109.25 60.25) (end 109.5 60.5) (width 0.2) (layer F.Cu) (net 2))
   (segment (start 109.25 59.55) (end 109.25 60.25) (width 0.2) (layer F.Cu) (net 2))
-  (segment (start 112.75 55.75) (end 112.5 55.5) (width 0.25) (layer F.Cu) (net 2))
-  (segment (start 112.5 55.5) (end 112 55.5) (width 0.25) (layer F.Cu) (net 2))
-  (segment (start 112.75 57.5) (end 112.75 55.75) (width 0.25) (layer F.Cu) (net 2))
-  (segment (start 112 58.25) (end 112.75 57.5) (width 0.25) (layer F.Cu) (net 2))
   (segment (start 111.25 52.75) (end 111.5 52.5) (width 0.25) (layer F.Cu) (net 2))
   (segment (start 111.5 52.5) (end 112 52.5) (width 0.25) (layer F.Cu) (net 2))
@@
   (segment (start 105.25 64.75) (end 105.25 64) (width 0.25) (layer F.Cu) (net 2))
   (via (at 112 58.5) (size 0.6) (drill 0.3) (layers F.Cu B.Cu) (net 2))
-  (segment (start 112 58.5) (end 112 58.25) (width 0.25) (layer F.Cu) (net 2))
   (segment (start 112 60) (end 112 58.5) (width 0.25) (layer F.Cu) (net 2))
-  (segment (start 107.25 58.5) (end 112 58.5) (width 0.25) (layer B.Cu) (net 2))
-  (segment (start 105.25 60.5) (end 107.25 58.5) (width 0.25) (layer B.Cu) (net 2))
   (segment (start 105.25 64) (end 105.25 60.5) (width 0.25) (layer B.Cu) (net 2))
+  (via (at 112 53.25) (size 0.6) (drill 0.3) (layers F.Cu B.Cu) (net 2))
+  (segment (start 112 52.5) (end 112 53.25) (width 0.25) (layer F.Cu) (net 2))
+  (segment (start 107.75 53.25) (end 105.25 55.75) (width 0.25) (layer B.Cu) (net 2))
+  (segment (start 105.25 55.75) (end 105.25 60.5) (width 0.25) (layer B.Cu) (net 2))
+  (segment (start 112 53.25) (end 107.75 53.25) (width 0.25) (layer B.Cu) (net 2))
+  (segment (start 105.25 58.5) (end 112 58.5) (width 0.25) (layer B.Cu) (net 2))
+  (segment (start 105.25 60.5) (end 105.25 58.5) (width 0.25) (layer B.Cu) (net 2))
   (segment (start 96.76 62) (end 96.69 62.07) (width 0.2) (layer F.Cu) (net 3))
   (segment (start 105 62) (end 96.76 62) (width 0.2) (layer F.Cu) (net 3))
@@
   (segment (start 103.51 63.25) (end 103.33 63.07) (width 0.2) (layer F.Cu) (net 9))
   (segment (start 105.25 63.25) (end 103.51 63.25) (width 0.2) (layer F.Cu) (net 9))
-  (segment (start 97.58 66.75) (end 120.17 66.75) (width 0.5) (layer F.Cu) (net 10))
-  (segment (start 98.923502 50.25) (end 120.17 50.25) (width 0.5) (layer F.Cu) (net 10))
-  (segment (start 97.58 50.25) (end 98.923502 50.25) (width 0.5) (layer F.Cu) (net 10))
   (segment (start 96.74 56) (end 96.69 55.95) (width 0.25) (layer F.Cu) (net 11))
   (segment (start 105 56) (end 96.74 56) (width 0.25) (layer F.Cu) (net 11))
@@
   (via (at 110.75 62) (size 0.6) (drill 0.3) (layers F.Cu B.Cu) (net 13))
   (segment (start 110.2 61.95) (end 110.7 61.95) (width 0.2) (layer F.Cu) (net 13))
-  (segment (start 110.75 62) (end 113 62) (width 0.2) (layer B.Cu) (net 13))
-  (via (at 113 62) (size 0.6) (drill 0.3) (layers F.Cu B.Cu) (net 13))
-  (segment (start 113 58) (end 113 62) (width 0.2) (layer F.Cu) (net 13))
-  (segment (start 116.25 54.75) (end 113 58) (width 0.2) (layer F.Cu) (net 13))
-  (segment (start 120.88 54.75) (end 116.25 54.75) (width 0.2) (layer F.Cu) (net 13))
-  (segment (start 121.06 54.93) (end 120.88 54.75) (width 0.2) (layer F.Cu) (net 13))
+  (via (at 113.75 62) (size 0.6) (drill 0.3) (layers F.Cu B.Cu) (net 13))
+  (segment (start 110.75 62) (end 113.75 62) (width 0.2) (layer B.Cu) (net 13))
+  (segment (start 113.75 57.25) (end 113.75 61.575736) (width 0.2) (layer F.Cu) (net 13))
+  (segment (start 113.75 61.575736) (end 113.75 62) (width 0.2) (layer F.Cu) (net 13))
+  (segment (start 121.06 54.93) (end 116.07 54.93) (width 0.2) (layer F.Cu) (net 13))
+  (segment (start 116.07 54.93) (end 113.75 57.25) (width 0.2) (layer F.Cu) (net 13))
   (segment (start 107.95 61.95) (end 108.3 61.95) (width 0.2) (layer F.Cu) (net 14))
   (segment (start 107 61) (end 107.95 61.95) (width 0.2) (layer F.Cu) (net 14))
@@
   (segment (start 108.3 61.95) (end 108.3 61.3) (width 0.2) (layer F.Cu) (net 14))
   (segment (start 108.3 61.3) (end 108.25 61.25) (width 0.2) (layer F.Cu) (net 14))
-  (segment (start 108.25 61.25) (end 113.75 61.25) (width 0.2) (layer B.Cu) (net 14))
-  (via (at 113.75 61.25) (size 0.6) (drill 0.3) (layers F.Cu B.Cu) (net 14))
-  (segment (start 113.75 58.25) (end 113.75 61.25) (width 0.2) (layer F.Cu) (net 14))
-  (segment (start 116 56) (end 113.75 58.25) (width 0.2) (layer F.Cu) (net 14))
-  (segment (start 119.23 56) (end 116 56) (width 0.2) (layer F.Cu) (net 14))
-  (segment (start 119.28 55.95) (end 119.23 56) (width 0.2) (layer F.Cu) (net 14))
+  (via (at 114.5 61.25) (size 0.6) (drill 0.3) (layers F.Cu B.Cu) (net 14))
+  (segment (start 116.05 55.95) (end 114.5 57.5) (width 0.2) (layer F.Cu) (net 14))
+  (segment (start 108.25 61.25) (end 114.5 61.25) (width 0.2) (layer B.Cu) (net 14))
+  (segment (start 119.28 55.95) (end 116.05 55.95) (width 0.2) (layer F.Cu) (net 14))
+  (segment (start 114.5 57.5) (end 114.5 60.825736) (width 0.2) (layer F.Cu) (net 14))
+  (segment (start 114.5 60.825736) (end 114.5 61.25) (width 0.2) (layer F.Cu) (net 14))
   (segment (start 107 60) (end 107.45 59.55) (width 0.2) (layer F.Cu) (net 15))
   (segment (start 107.45 59.55) (end 108.3 59.55) (width 0.2) (layer F.Cu) (net 15))
@@
   (segment (start 108.3 60.2) (end 108.25 60.25) (width 0.2) (layer F.Cu) (net 15))
   (segment (start 108.3 59.55) (end 108.3 60.2) (width 0.2) (layer F.Cu) (net 15))
-  (segment (start 108.25 60.25) (end 114.5 60.25) (width 0.2) (layer B.Cu) (net 15))
-  (via (at 114.5 60.25) (size 0.6) (drill 0.3) (layers F.Cu B.Cu) (net 15))
-  (segment (start 114.5 58.5) (end 114.5 60.25) (width 0.2) (layer F.Cu) (net 15))
-  (segment (start 116.03 56.97) (end 114.5 58.5) (width 0.2) (layer F.Cu) (net 15))
+  (via (at 115.249992 60.25) (size 0.6) (drill 0.3) (layers F.Cu B.Cu) (net 15))
+  (segment (start 108.25 60.25) (end 115.249992 60.25) (width 0.2) (layer B.Cu) (net 15))
+  (segment (start 115.249992 59.825736) (end 115.249992 60.25) (width 0.2) (layer F.Cu) (net 15))
   (segment (start 121.06 56.97) (end 116.03 56.97) (width 0.2) (layer F.Cu) (net 15))
+  (segment (start 116.03 56.97) (end 115.249992 57.750008) (width 0.2) (layer F.Cu) (net 15))
+  (segment (start 115.249992 57.750008) (end 115.249992 59.825736) (width 0.2) (layer F.Cu) (net 15))
   (segment (start 110.2 58.05) (end 110.2 57.45) (width 0.2) (layer F.Cu) (net 16))
   (segment (start 110 58.25) (end 110.2 58.05) (width 0.2) (layer F.Cu) (net 16))
@@
   (segment (start 110.7 59.55) (end 110.75 59.5) (width 0.2) (layer F.Cu) (net 18))
   (segment (start 110.2 59.55) (end 110.7 59.55) (width 0.2) (layer F.Cu) (net 18))
-  (via (at 115.25 60) (size 0.6) (drill 0.3) (layers F.Cu B.Cu) (net 18))
-  (segment (start 119.25 60) (end 115.25 60) (width 0.2) (layer F.Cu) (net 18))
+  (via (at 116.75 60) (size 0.6) (drill 0.3) (layers F.Cu B.Cu) (net 18))
+  (segment (start 110.75 59.5) (end 116.25 59.5) (width 0.2) (layer B.Cu) (net 18))
+  (segment (start 116.25 59.5) (end 116.450001 59.700001) (width 0.2) (layer B.Cu) (net 18))
+  (segment (start 116.450001 59.700001) (end 116.75 60) (width 0.2) (layer B.Cu) (net 18))
+  (segment (start 119.25 60) (end 116.75 60) (width 0.2) (layer F.Cu) (net 18))
   (segment (start 119.28 60.03) (end 119.25 60) (width 0.2) (layer F.Cu) (net 18))
-  (segment (start 115 59.75) (end 115.25 60) (width 0.2) (layer B.Cu) (net 18))
-  (segment (start 114.75 59.5) (end 115 59.75) (width 0.2) (layer B.Cu) (net 18))
-  (segment (start 110.75 59.5) (end 114.75 59.5) (width 0.2) (layer B.Cu) (net 18))
   (segment (start 107.95 55.05) (end 108.3 55.05) (width 0.25) (layer F.Cu) (net 19))
   (segment (start 107 56) (end 107.95 55.05) (width 0.25) (layer F.Cu) (net 19))
@@
     (connect_pads (clearance 0.2))
     (min_thickness 0.2)
+    (fill yes (arc_segments 32) (thermal_gap 0.2) (thermal_bridge_width 0.25))
+    (polygon
+      (pts
+        (xy 90.75 47.5) (xy 157.5 47.5) (xy 157.5 69.5) (xy 90.75 69.5)
+      )
+    )
+  )
+  (zone (net 10) (net_name 13) (layer B.Cu) (hatch edge 0.508)
+    (connect_pads (clearance 0.2))
+    (min_thickness 0.2)

Commit message: parts
Other:
- board size 66.8 x 22 mm -> 36.2 x 22 mm
Changed lines of the file:
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@@
   (general
     (thickness 1.6)
-    (drawings 4)
+    (drawings 8)
     (tracks 158)
     (zones 0)
@@
   )
   (setup
-    (last_trace_width 0.25)
+    (last_trace_width 0.2)
     (user_trace_width 0.2)
     (user_trace_width 0.25)
@@
     (add_net 8_8)
     (add_net GND)
-    (add_net "Net-(J1-Pad10)")
     (add_net "Net-(J1-Pad12)")
-    (add_net "Net-(J1-Pad9)")
-    (add_net "Net-(J2-Pad10)")
-    (add_net "Net-(J2-Pad11)")
     (add_net "Net-(J2-Pad12)")
-    (add_net "Net-(J2-Pad9)")
   )
   (net_class PE ""
@@
     )
   )
-  (gr_line (start 90.75 47.5) (end 157.5 47.5) (layer Edge.Cuts) (width 0.15))
-  (gr_line (start 90.75 69.5) (end 90.75 47.5) (layer Edge.Cuts) (width 0.15))
-  (gr_line (start 157.5 69.5) (end 90.75 69.5) (layer Edge.Cuts) (width 0.15))
-  (gr_line (start 157.5 47.5) (end 157.5 69.5) (layer Edge.Cuts) (width 0.15))
+  (gr_arc (start 91.75 68.5) (end 90.75 68.5) (angle -90) (layer Edge.Cuts) (width 0.15))
+  (gr_arc (start 91.75 48.5) (end 91.75 47.5) (angle -90) (layer Edge.Cuts) (width 0.15))
+  (gr_arc (start 126 48.5) (end 127 48.5) (angle -90) (layer Edge.Cuts) (width 0.15))
+  (gr_arc (start 126 68.5) (end 126 69.5) (angle -90) (layer Edge.Cuts) (width 0.15))
+  (gr_line (start 91.75 47.5) (end 126 47.5) (layer Edge.Cuts) (width 0.15))
+  (gr_line (start 90.75 68.5) (end 90.75 48.5) (layer Edge.Cuts) (width 0.15))
+  (gr_line (start 126 69.5) (end 91.75 69.5) (layer Edge.Cuts) (width 0.15))
+  (gr_line (start 127 48.5) (end 127 68.5) (layer Edge.Cuts) (width 0.15))
   (segment (start 111.5 55.5) (end 112 55.5) (width 0.2) (layer F.Cu) (net 2))
   (segment (start 111 56) (end 111.5 55.5) (width 0.2) (layer F.Cu) (net 2))
@@
     (polygon
       (pts
-        (xy 90.75 47.5) (xy 157.5 47.5) (xy 157.5 69.5) (xy 90.75 69.5)
+        (xy 90.75 47.5) (xy 127 47.5) (xy 127 69.5) (xy 90.75 69.5)
       )
     )
@@
     (polygon
       (pts
-        (xy 90.75 47.5) (xy 157.5 47.5) (xy 157.5 69.5) (xy 90.75 69.5)
+        (xy 90.75 47.5) (xy 127 47.5) (xy 127 69.5) (xy 90.75 69.5)
       )
     )

Commit message: jlc export
Parts:
- renumbered C11 to C201, C1 to C202, J1 to J201, J2 to J202, R1 to R201, R2 to R202, U11 to U201, U1 to U202, U6 to U203, U2 to U204, U3 to U205, U4 to U206
