File: cmc/pcb.sch (KiCad schematic (older format))
At the start: 12 parts, among them J1 RJ45_LED, J2 RJ45_LED, U1 CMC, U11 CMC, U2 USBLC6-4SC6, U3 CMC, U4 CMC, U6 USBLC6-4SC6

Commit message: parts
Parts:
- C1, C11: LCSC (none) -> C14663
- R1, R2: LCSC (none) -> C23204
- U1, U11, U3, U4: LCSC (none) -> C80529
- U2, U6: LCSC (none) -> C111212
Changed lines of the file:
@@
 F 2 "stmbl:SOT-23-6" H 5450 2950 50  0001 C CNN
 F 3 "" H 4900 2850 50  0001 C CNN
+F 4 " C111212" H 5150 2500 50  0001 C CNN "LCSC"
 	1    5150 2500
 	1    0    0    -1
@@
 F 2 "stmbl:C_0603" H 7215 2409 50  0001 L CNN
 F 3 "" H 7100 2500 50  0001 C CNN
+F 4 "C14663" H 7100 2500 50  0001 C CNN "LCSC"
 	1    7100 2500
 	1    0    0    -1
@@
 F 3 "" H 3750 2500 60  0001 C CNN
 F 4 "DLW21HN900SQ2L" H 3750 2500 50  0001 C CNN "Manufacturer No"
+F 5 "C80529" H 3750 2500 50  0001 C CNN "LCSC"
 	1    3750 2500
 	-1   0    0    1
@@
 F 3 "" H 6550 2500 60  0001 C CNN
 F 4 "DLW21HN900SQ2L" H 6550 2500 50  0001 C CNN "Manufacturer No"
+F 5 "C80529" H 6550 2500 50  0001 C CNN "LCSC"
 	1    6550 2500
 	1    0    0    1
@@
 F 2 "stmbl:SOT-23-6" H 5450 4000 50  0001 C CNN
 F 3 "" H 4900 3900 50  0001 C CNN
+F 4 " C111212" H 5150 3550 50  0001 C CNN "LCSC"
 	1    5150 3550
 	1    0    0    -1
@@
 F 2 "stmbl:C_0603" H 7215 3459 50  0001 L CNN
 F 3 "" H 7100 3550 50  0001 C CNN
+F 4 "C14663" H 7100 3550 50  0001 C CNN "LCSC"
 	1    7100 3550
 	1    0    0    -1
@@
 F 3 "" H 3750 3550 60  0001 C CNN
 F 4 "DLW21HN900SQ2L" H 3750 3550 50  0001 C CNN "Manufacturer No"
+F 5 "C80529" H 3750 3550 50  0001 C CNN "LCSC"
 	1    3750 3550
 	-1   0    0    1
@@
 F 3 "" H 6550 3550 60  0001 C CNN
 F 4 "DLW21HN900SQ2L" H 6550 3550 50  0001 C CNN "Manufacturer No"
+F 5 "C80529" H 6550 3550 50  0001 C CNN "LCSC"
 	1    6550 3550
 	1    0    0    1
@@
 F 2 "stmbl:R_0603" V 1080 2150 50  0001 C CNN
 F 3 "" H 1150 2150 50  0001 C CNN
+F 4 "C23204" H 1150 2150 50  0001 C CNN "LCSC"
 	1    1150 2150
 	0    1    1    0
@@
 F 2 "stmbl:R_0603" V 1080 3800 50  0001 C CNN
 F 3 "" H 1150 3800 50  0001 C CNN
+F 4 "C23204" H 1150 3800 50  0001 C CNN "LCSC"
 	1    1150 3800
 	0    1    1    0

Commit message: jlc export
Parts:
- U203: renamed from U6; LCSC C111212 -> C111212
- U204: renamed from U2; LCSC C111212 -> C111212
- renumbered C11 to C201, C1 to C202, J1 to J201, J2 to J202, R1 to R201, R2 to R202, U11 to U201, U1 to U202, U3 to U205, U4 to U206
Changed lines of the file:
@@
 $EndDescr
 $Comp
-L stmbl:RJ45_LED J1
+L stmbl:RJ45_LED J201
 U 1 1 5E3EE2C2
 P 1900 2550
-F 0 "J1" V 1275 2550 50  0000 C CNN
+F 0 "J201" V 1275 2550 50  0000 C CNN
 F 1 "RJ45_LED" V 1366 2550 50  0000 C CNN
 F 2 "stmbl:RJ45_LED" V 1359 2550 60  0001 C CNN
@@
 $EndComp
 $Comp
-L stmbl:USBLC6-4SC6 U6
+L stmbl:USBLC6-4SC6 U203
 U 1 1 5E44C1CC
 P 5150 2500
-F 0 "U6" H 5150 3067 50  0000 C CNN
+F 0 "U203" H 5150 3067 50  0000 C CNN
 F 1 "USBLC6-4SC6" H 5150 2976 50  0000 C CNN
 F 2 "stmbl:SOT-23-6" H 5450 2950 50  0001 C CNN
 F 3 "" H 4900 2850 50  0001 C CNN
-F 4 " C111212" H 5150 2500 50  0001 C CNN "LCSC"
+F 4 "C111212" H 5150 2500 50  0001 C CNN "LCSC"
 	1    5150 2500
 	1    0    0    -1
 $EndComp
 $Comp
-L stmbl:C C11
+L stmbl:C C201
 U 1 1 5E44E6F8
 P 7100 2500
-F 0 "C11" H 7215 2546 50  0000 L CNN
+F 0 "C201" H 7215 2546 50  0000 L CNN
 F 1 "100n" H 7215 2455 50  0000 L CNN
 F 2 "stmbl:C_0603" H 7215 2409 50  0001 L CNN
@@
 	5750 2500 5650 2500
 $Comp
-L stmbl:+3.3V #PWR038
+L stmbl:+3.3V #PWR0207
 U 1 1 5E451F3C
 P 5750 2500
-F 0 "#PWR038" H 5750 2350 50  0001 C CNN
+F 0 "#PWR0207" H 5750 2350 50  0001 C CNN
 F 1 "+3.3V" V 5765 2628 50  0000 L CNN
 F 2 "" H 5750 2500 50  0001 C CNN
@@
 $EndComp
 $Comp
-L stmbl:+3.3V #PWR033
+L stmbl:+3.3V #PWR0209
 U 1 1 5E452F59
 P 7100 2250
-F 0 "#PWR033" H 7100 2100 50  0001 C CNN
+F 0 "#PWR0209" H 7100 2100 50  0001 C CNN
 F 1 "+3.3V" H 7115 2423 50  0000 C CNN
 F 2 "" H 7100 2250 50  0001 C CNN
@@
 $EndComp
 $Comp
-L stmbl:GND #PWR034
+L stmbl:GND #PWR0210
 U 1 1 5E453228
 P 7100 2750
-F 0 "#PWR034" H 7100 2500 50  0001 C CNN
+F 0 "#PWR0210" H 7100 2500 50  0001 C CNN
 F 1 "GND" H 7105 2577 50  0000 C CNN
 F 2 "" H 7100 2750 50  0001 C CNN
@@
 	7100 2350 7100 2250
 $Comp
-L stmbl:GND #PWR031
+L stmbl:GND #PWR0205
 U 1 1 5E4560FE
 P 4550 2500
-F 0 "#PWR031" H 4550 2250 50  0001 C CNN
+F 0 "#PWR0205" H 4550 2250 50  0001 C CNN
 F 1 "GND" V 4555 2372 50  0000 R CNN
 F 2 "" H 4550 2500 50  0001 C CNN
@@
 6
 $Comp
-L stmbl:CMC U11
+L stmbl:CMC U201
 U 1 1 5E354A2F
 P 3750 2500
-F 0 "U11" H 3750 2797 60  0000 C CNN
+F 0 "U201" H 3750 2797 60  0000 C CNN
 F 1 "CMC" H 3750 2691 60  0000 C CNN
 F 2 "stmbl:CMC_0805" H 3750 2500 60  0001 C CNN
@@
 	1900 3200 1900 3300
 $Comp
-L stmbl:RJ45_LED J2
+L stmbl:RJ45_LED J202
 U 1 1 5E7A8F61
 P 1900 4200
-F 0 "J2" V 1275 4200 50  0000 C CNN
+F 0 "J202" V 1275 4200 50  0000 C CNN
 F 1 "RJ45_LED" V 1366 4200 50  0000 C CNN
 F 2 "stmbl:RJ45_LED" V 1359 4200 60  0001 C CNN
@@
 	4050 2300 4150 2300
 $Comp
-L stmbl:CMC U3
+L stmbl:CMC U205
 U 1 1 5E7C2940
 P 6550 2500
-F 0 "U3" H 6550 2797 60  0000 C CNN
+F 0 "U205" H 6550 2797 60  0000 C CNN
 F 1 "CMC" H 6550 2691 60  0000 C CNN
 F 2 "stmbl:CMC_0805" H 6550 2500 60  0001 C CNN
@@
 Connection ~ 6150 2300
 $Comp
-L stmbl:USBLC6-4SC6 U2
+L stmbl:USBLC6-4SC6 U204
 U 1 1 5E7C94CA
 P 5150 3550
-F 0 "U2" H 5150 4117 50  0000 C CNN
+F 0 "U204" H 5150 4117 50  0000 C CNN
 F 1 "USBLC6-4SC6" H 5150 4026 50  0000 C CNN
 F 2 "stmbl:SOT-23-6" H 5450 4000 50  0001 C CNN
 F 3 "" H 4900 3900 50  0001 C CNN
-F 4 " C111212" H 5150 3550 50  0001 C CNN "LCSC"
+F 4 "C111212" H 5150 3550 50  0001 C CNN "LCSC"
 	1    5150 3550
 	1    0    0    -1
 $EndComp
 $Comp
-L stmbl:C C1
+L stmbl:C C202
 U 1 1 5E7C94D4
 P 7100 3550
-F 0 "C1" H 7215 3596 50  0000 L CNN
+F 0 "C202" H 7215 3596 50  0000 L CNN
 F 1 "100n" H 7215 3505 50  0000 L CNN
 F 2 "stmbl:C_0603" H 7215 3459 50  0001 L CNN
@@
 	5750 3550 5650 3550
 $Comp
-L stmbl:+3.3V #PWR0101
+L stmbl:+3.3V #PWR0208
 U 1 1 5E7C94DF
 P 5750 3550
-F 0 "#PWR0101" H 5750 3400 50  0001 C CNN
+F 0 "#PWR0208" H 5750 3400 50  0001 C CNN
 F 1 "+3.3V" V 5765 3678 50  0000 L CNN
 F 2 "" H 5750 3550 50  0001 C CNN
@@
 $EndComp
 $Comp
-L stmbl:+3.3V #PWR0102
+L stmbl:+3.3V #PWR0211
 U 1 1 5E7C94E9
 P 7100 3300
-F 0 "#PWR0102" H 7100 3150 50  0001 C CNN
+F 0 "#PWR0211" H 7100 3150 50  0001 C CNN
 F 1 "+3.3V" H 7115 3473 50  0000 C CNN
 F 2 "" H 7100 3300 50  0001 C CNN
@@
 $EndComp
 $Comp
-L stmbl:GND #PWR0103
+L stmbl:GND #PWR0212
 U 1 1 5E7C94F3
 P 7100 3800
-F 0 "#PWR0103" H 7100 3550 50  0001 C CNN
+F 0 "#PWR0212" H 7100 3550 50  0001 C CNN
 F 1 "GND" H 7105 3627 50  0000 C CNN
 F 2 "" H 7100 3800 50  0001 C CNN
@@
 	7100 3400 7100 3300
 $Comp
-L stmbl:GND #PWR0104
+L stmbl:GND #PWR0206
 U 1 1 5E7C94FF
 P 4550 3550
-F 0 "#PWR0104" H 4550 3300 50  0001 C CNN
+F 0 "#PWR0206" H 4550 3300 50  0001 C CNN
 F 1 "GND" V 4555 3422 50  0000 R CNN
 F 2 "" H 4550 3550 50  0001 C CNN
@@
 	4550 3550 4650 3550
 $Comp
-L stmbl:CMC U1
+L stmbl:CMC U202
 U 1 1 5E7C950B
 P 3750 3550
-F 0 "U1" H 3750 3847 60  0000 C CNN
+F 0 "U202" H 3750 3847 60  0000 C CNN
 F 1 "CMC" H 3750 3741 60  0000 C CNN
 F 2 "stmbl:CMC_0805" H 3750 3550 60  0001 C CNN
@@
 	4050 3350 4150 3350
 $Comp
-L stmbl:CMC U4
+L stmbl:CMC U206
 U 1 1 5E7C9526
 P 6550 3550
-F 0 "U4" H 6550 3847 60  0000 C CNN
+F 0 "U206" H 6550 3847 60  0000 C CNN
 F 1 "CMC" H 6550 3741 60  0000 C CNN
 F 2 "stmbl:CMC_0805" H 6550 3550 60  0001 C CNN
@@
 	900  2150 1000 2150
 $Comp
-L stmbl:+3.3V #PWR0106
+L stmbl:+3.3V #PWR0201
 U 1 1 5E82A08F
 P 900 2150
-F 0 "#PWR0106" H 900 2000 50  0001 C CNN
+F 0 "#PWR0201" H 900 2000 50  0001 C CNN
 F 1 "+3.3V" H 915 2323 50  0000 C CNN
 F 2 "" H 900 2150 50  0001 C CNN
@@
 $EndComp
 $Comp
-L stmbl:R R1
+L stmbl:R R201
 U 1 1 5E8299DE
 P 1150 2150
-F 0 "R1" V 943 2150 50  0000 C CNN
+F 0 "R201" V 943 2150 50  0000 C CNN
 F 1 "560" V 1034 2150 50  0000 C CNN
 F 2 "stmbl:R_0603" V 1080 2150 50  0001 C CNN
@@
 $EndComp
 $Comp
-L stmbl:GND #PWR0105
+L stmbl:GND #PWR0203
 U 1 1 5E828CAF
 P 1300 2250
-F 0 "#PWR0105" H 1300 2000 50  0001 C CNN
+F 0 "#PWR0203" H 1300 2000 50  0001 C CNN
 F 1 "GND" H 1305 2077 50  0000 C CNN
 F 2 "" H 1300 2250 50  0001 C CNN
@@
 	900  3800 1000 3800
 $Comp
-L stmbl:+3.3V #PWR0107
+L stmbl:+3.3V #PWR0202
 U 1 1 5E8334FE
 P 900 3800
-F 0 "#PWR0107" H 900 3650 50  0001 C CNN
+F 0 "#PWR0202" H 900 3650 50  0001 C CNN
 F 1 "+3.3V" H 915 3973 50  0000 C CNN
 F 2 "" H 900 3800 50  0001 C CNN
@@
 $EndComp
 $Comp
-L stmbl:R R2
+L stmbl:R R202
 U 1 1 5E833508
 P 1150 3800
-F 0 "R2" V 943 3800 50  0000 C CNN
+F 0 "R202" V 943 3800 50  0000 C CNN
 F 1 "560" V 1034 3800 50  0000 C CNN
 F 2 "stmbl:R_0603" V 1080 3800 50  0001 C CNN
@@
 $EndComp
 $Comp
-L stmbl:GND #PWR0108
+L stmbl:GND #PWR0204
 U 1 1 5E833512
 P 1300 3900
-F 0 "#PWR0108" H 1300 3650 50  0001 C CNN
+F 0 "#PWR0204" H 1300 3650 50  0001 C CNN
 F 1 "GND" H 1305 3727 50  0000 C CNN
 F 2 "" H 1300 3900 50  0001 C CNN
