File: hx711/hx711.sch (KiCad schematic (older format))
At the start: 14 parts, among them U8 HX711

Commit message: hx711
Parts:
- C15, C16, C17, C18, C19: footprint stmbl:C0603 -> stmbl:C_0603
- JP1, JP2: footprint (none) -> stmbl:0603_jumper
- R4, R5, R6, R7, R8, R9: footprint stmbl:R0603 -> stmbl:R_0603
- U8: footprint (none) -> stmbl:SOIC-16
Changed lines of the file:
@@
 EESchema Schematic File Version 4
+LIBS:pcb-cache
 EELAYER 30 0
 EELAYER END
 $Descr A4 11693 8268
 encoding utf-8
-Sheet 2 3
+Sheet 3 3
 Title ""
 Date ""
@@
 F 0 "U9" H 4500 3947 60  0000 C CNN
 F 1 "HX711" H 4500 3841 60  0000 C CNN
-F 2 "" H 4500 3300 60  0001 C CNN
+F 2 "stmbl:SOIC-16" H 4500 3300 60  0001 C CNN
 F 3 "" H 4500 3300 60  0001 C CNN
 	1    4500 3300
@@
 F 0 "R12" V 6157 2700 50  0000 C CNN
 F 1 "100" V 6066 2700 50  0000 C CNN
-F 2 "stmbl:R0603" H 6020 2609 50  0001 L CNN
+F 2 "stmbl:R_0603" H 6020 2609 50  0001 L CNN
 F 3 "" H 5950 2700 50  0001 C CNN
 	1    5950 2700
@@
 F 0 "R13" V 6157 2900 50  0000 C CNN
 F 1 "100" V 6066 2900 50  0000 C CNN
-F 2 "stmbl:R0603" H 6020 2809 50  0001 L CNN
+F 2 "stmbl:R_0603" H 6020 2809 50  0001 L CNN
 F 3 "" H 5950 2900 50  0001 C CNN
 	1    5950 2900
@@
 F 0 "C23" V 5198 2900 50  0000 C CNN
 F 1 "100n" V 5289 2900 50  0000 C CNN
-F 2 "stmbl:C0603" H 5565 2809 50  0001 L CNN
+F 2 "stmbl:C_0603" H 5565 2809 50  0001 L CNN
 F 3 "" H 5450 2900 50  0001 C CNN
 	1    5450 2900
@@
 F 0 "C24" V 5198 3300 50  0000 C CNN
 F 1 "100n" V 5289 3300 50  0000 C CNN
-F 2 "stmbl:C0603" H 5565 3209 50  0001 L CNN
+F 2 "stmbl:C_0603" H 5565 3209 50  0001 L CNN
 F 3 "" H 5450 3300 50  0001 C CNN
 	1    5450 3300
@@
 F 0 "R14" V 6157 3300 50  0000 C CNN
 F 1 "100" V 6066 3300 50  0000 C CNN
-F 2 "stmbl:R0603" H 6020 3209 50  0001 L CNN
+F 2 "stmbl:R_0603" H 6020 3209 50  0001 L CNN
 F 3 "" H 5950 3300 50  0001 C CNN
 	1    5950 3300
@@
 F 0 "R15" V 6157 3500 50  0000 C CNN
 F 1 "100" V 6066 3500 50  0000 C CNN
-F 2 "stmbl:R0603" H 6020 3409 50  0001 L CNN
+F 2 "stmbl:R_0603" H 6020 3409 50  0001 L CNN
 F 3 "" H 5950 3500 50  0001 C CNN
 	1    5950 3500
@@
 F 0 "R11" V 5457 3800 50  0000 C CNN
 F 1 "1k" V 5366 3800 50  0000 C CNN
-F 2 "stmbl:R0603" H 5320 3709 50  0001 L CNN
+F 2 "stmbl:R_0603" H 5320 3709 50  0001 L CNN
 F 3 "" H 5250 3800 50  0001 C CNN
 	1    5250 3800
@@
 F 0 "JP4" H 5250 4093 50  0000 C CNN
 F 1 "Jumper_NO_Small" H 5260 3940 50  0001 C CNN
-F 2 "" H 5250 4000 50  0000 C CNN
+F 2 "stmbl:0603_jumper" H 5250 4000 50  0001 C CNN
 F 3 "" H 5250 4000 50  0000 C CNN
 	1    5250 4000
@@
 F 0 "C21" H 2635 2954 50  0000 R CNN
 F 1 "100n" H 2635 3045 50  0000 R CNN
-F 2 "stmbl:C0603" H 2865 2909 50  0001 L CNN
+F 2 "stmbl:C_0603" H 2865 2909 50  0001 L CNN
 F 3 "" H 2750 3000 50  0001 C CNN
 	1    2750 3000
@@
 F 0 "C20" H 2235 2954 50  0000 R CNN
 F 1 "100n" H 2235 3045 50  0000 R CNN
-F 2 "stmbl:C0603" H 2465 2909 50  0001 L CNN
+F 2 "stmbl:C_0603" H 2465 2909 50  0001 L CNN
 F 3 "" H 2350 3000 50  0001 C CNN
 	1    2350 3000
@@
 F 0 "C22" V 4002 3800 50  0000 C CNN
 F 1 "20pf" V 3911 3800 50  0000 C CNN
-F 2 "stmbl:C0603" H 3865 3709 50  0001 L CNN
+F 2 "stmbl:C_0603" H 3865 3709 50  0001 L CNN
 F 3 "" H 3750 3800 50  0001 C CNN
 	1    3750 3800
@@
 F 0 "JP3" H 3750 4143 50  0000 C CNN
 F 1 "Jumper_NO_Small" H 3760 3990 50  0001 C CNN
-F 2 "" H 3750 4050 50  0000 C CNN
+F 2 "stmbl:0603_jumper" H 3750 4050 50  0001 C CNN
 F 3 "" H 3750 4050 50  0000 C CNN
 	1    3750 4050
@@
 F 0 "R10" V 3507 3800 50  0000 C CNN
 F 1 "1k" V 3416 3800 50  0000 C CNN
-F 2 "stmbl:R0603" H 3370 3709 50  0001 L CNN
+F 2 "stmbl:R_0603" H 3370 3709 50  0001 L CNN
 F 3 "" H 3300 3800 50  0001 C CNN
 	1    3300 3800

Commit message: parts
Parts:
- C15, C16, C18, C19: LCSC (none) -> C14663
- C17: LCSC (none) -> C1648
- R4, R5: LCSC (none) -> C21190
- R6, R7, R8, R9: value 100 -> 120; LCSC (none) -> C22787
- U8: LCSC (none) -> C43656
Changed lines of the file:
@@
 F 2 "stmbl:SOIC-16" H 4500 3300 60  0001 C CNN
 F 3 "" H 4500 3300 60  0001 C CNN
+F 4 "C43656" H 4500 3300 50  0001 C CNN "LCSC"
 	1    4500 3300
 	1    0    0    -1
@@
 AR Path="/5E43BA91/5E430A27" Ref="R12"  Part="1"
 F 0 "R12" V 6157 2700 50  0000 C CNN
-F 1 "100" V 6066 2700 50  0000 C CNN
+F 1 "120" V 6066 2700 50  0000 C CNN
 F 2 "stmbl:R_0603" H 6020 2609 50  0001 L CNN
 F 3 "" H 5950 2700 50  0001 C CNN
+F 4 "C22787" H 5950 2700 50  0001 C CNN "LCSC"
 	1    5950 2700
 	0    -1   -1   0
@@
 AR Path="/5E43BA91/5E430A46" Ref="R13"  Part="1"
 F 0 "R13" V 6157 2900 50  0000 C CNN
-F 1 "100" V 6066 2900 50  0000 C CNN
+F 1 "120" V 6066 2900 50  0000 C CNN
 F 2 "stmbl:R_0603" H 6020 2809 50  0001 L CNN
 F 3 "" H 5950 2900 50  0001 C CNN
+F 4 "C22787" H 5950 2900 50  0001 C CNN "LCSC"
 	1    5950 2900
 	0    -1   -1   0
@@
 F 2 "stmbl:C_0603" H 5565 2809 50  0001 L CNN
 F 3 "" H 5450 2900 50  0001 C CNN
+F 4 "C14663" H 5450 2900 50  0001 C CNN "LCSC"
 	1    5450 2900
 	0    1    1    0
@@
 F 2 "stmbl:C_0603" H 5565 3209 50  0001 L CNN
 F 3 "" H 5450 3300 50  0001 C CNN
+F 4 "C14663" H 5450 3300 50  0001 C CNN "LCSC"
 	1    5450 3300
 	0    1    1    0
@@
 AR Path="/5E43BA91/5E430A62" Ref="R14"  Part="1"
 F 0 "R14" V 6157 3300 50  0000 C CNN
-F 1 "100" V 6066 3300 50  0000 C CNN
+F 1 "120" V 6066 3300 50  0000 C CNN
 F 2 "stmbl:R_0603" H 6020 3209 50  0001 L CNN
 F 3 "" H 5950 3300 50  0001 C CNN
+F 4 "C22787" H 5950 3300 50  0001 C CNN "LCSC"
 	1    5950 3300
 	0    -1   -1   0
@@
 AR Path="/5E43BA91/5E430A68" Ref="R15"  Part="1"
 F 0 "R15" V 6157 3500 50  0000 C CNN
-F 1 "100" V 6066 3500 50  0000 C CNN
+F 1 "120" V 6066 3500 50  0000 C CNN
 F 2 "stmbl:R_0603" H 6020 3409 50  0001 L CNN
 F 3 "" H 5950 3500 50  0001 C CNN
+F 4 "C22787" H 5950 3500 50  0001 C CNN "LCSC"
 	1    5950 3500
 	0    -1   -1   0
@@
 F 2 "stmbl:R_0603" H 5320 3709 50  0001 L CNN
 F 3 "" H 5250 3800 50  0001 C CNN
+F 4 "C21190" H 5250 3800 50  0001 C CNN "LCSC"
 	1    5250 3800
 	0    -1   -1   0
@@
 F 2 "stmbl:C_0603" H 2865 2909 50  0001 L CNN
 F 3 "" H 2750 3000 50  0001 C CNN
+F 4 "C14663" H 2750 3000 50  0001 C CNN "LCSC"
 	1    2750 3000
 	-1   0    0    1
@@
 F 2 "stmbl:C_0603" H 2465 2909 50  0001 L CNN
 F 3 "" H 2350 3000 50  0001 C CNN
+F 4 "C14663" H 2350 3000 50  0001 C CNN "LCSC"
 	1    2350 3000
 	-1   0    0    1
@@
 F 2 "stmbl:C_0603" H 3865 3709 50  0001 L CNN
 F 3 "" H 3750 3800 50  0001 C CNN
+F 4 "C1648" H 3750 3800 50  0001 C CNN "LCSC"
 	1    3750 3800
 	0    -1   -1   0
@@
 F 2 "stmbl:R_0603" H 3370 3709 50  0001 L CNN
 F 3 "" H 3300 3800 50  0001 C CNN
+F 4 "C21190" H 3300 3800 50  0001 C CNN "LCSC"
 	1    3300 3800
 	0    -1   -1   0

Commit message: jlc export
Parts:
- renumbered C15 to C316, C16 to C317, C17 to C318, C18 to C319, C19 to C320, JP1 to JP301, JP2 to JP302, R4 to R305, R5 to R306, R6 to R307, R7 to R308, R8 to R309, R9 to R310, U8 to U313
