File: hx711/pcb.kicad_pcb (KiCad board)
At the start: 4 copper layers, 56.8 x 22 mm, 59 parts, among them J1 RJ45_LED, J2 CONN_02X03_Odd_Even, J3 CONN_02X03_Odd_Even, J4 CONN_02X03_Odd_Even, J5 CONN_02X03_Odd_Even, U1 sp485, U2 RS485, U3 RS485, U4 20M, U5 MIC55, U6 USBLC6-4SC6, U7 USBLC6-4SC6, U8 HX711, U9 HX711

Commit message: hx711
Parts:
- added C25: 100p, stmbl:C_0603, F.Cu at (116.5, 67.8)
- added U10: CMC, stmbl:CMC_0805, F.Cu at (103.0, 49.0)
- added U11: CMC, stmbl:CMC_0805, F.Cu at (136.8, 67.2)
- added U12: CMC, stmbl:CMC_0805, F.Cu at (136.8, 60.2)
- added U13: CMC, stmbl:CMC_0805, F.Cu at (136.8, 56.8)
- added U14: CMC, stmbl:CMC_0805, F.Cu at (136.8, 49.8)
- J2, J3, J4, J5: value CONN_02X03_Odd_Even -> CONN_01X05; footprint stmbl:Pin_Header_RM2.54_2x3_UP -> stmbl:Pin_Header_RM2.54_1x5_UP
- U5: value MIC55 -> LDO
- moved C14 2.46 mm to (118.5, 64.0), turned to 0 degrees
- moved L1 2.24 mm to (116.5, 64.8)
- moved J3 2.06 mm to (139.5, 60.5)
- moved J5 2.06 mm to (139.5, 50.0)
- moved C9 1.50 mm to (118.2, 67.5)
- moved C12 1.03 mm to (117.0, 62.2), turned to 0 degrees
- moved J2 0.90 mm to (139.5, 67.0)
- moved J4 0.90 mm to (139.5, 56.5)
- moved U5 0.50 mm to (112.2, 67.2)
- moved C10 0.50 mm to (115.0, 67.0)
- moved C8 0.50 mm to (109.5, 67.0)
- moved C1 0.25 mm to (100.5, 67.8)
- moved C2 0.25 mm to (106.0, 64.8)
- moved C3 0.25 mm to (106.0, 59.5)
- moved C4 0.25 mm to (106.0, 54.2)
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Connections:
- J1 pad 7: +5V -> Net-(J1-Pad7)
- J1 pad 8: GND -> Net-(J1-Pad8)
- J2 pad 2: A1+ -> Net-(J2-Pad2)
- J2 pad 3: A1- -> Net-(J2-Pad3)
- J2 pad 5: GND -> GNDS
- J3 pad 2: B1+ -> Net-(J3-Pad2)
- J3 pad 3: B1- -> Net-(J3-Pad3)
- J3 pad 5: GND -> GNDS
- J4 pad 2: A2+ -> Net-(J4-Pad2)
- J4 pad 3: A2- -> Net-(J4-Pad3)
- J4 pad 5: GND -> GNDS
- J5 pad 2: B2+ -> Net-(J5-Pad2)
- J5 pad 3: B2- -> Net-(J5-Pad3)
- J5 pad 5: GND -> GNDS
- U2 pad 1: (no net) -> SCK
- U2 pad 4: SCK -> (no net)
- U5 pad 3: (no net) -> +5V
- U5 pad 4: (no net) -> Net-(C25-Pad2)
Other:
- board size 56.8 x 22 mm -> 66.8 x 22 mm
- board text added: "3.3V A+B A-B GND SHD"

Commit message: hx711
Parts:
- moved C9 17.6 mm to (116.5, 50.0)
- moved C10 17.5 mm to (114.8, 49.5)
- moved C5 17.5 mm to (107.5, 50.0)
- moved C7 17.5 mm to (105.5, 50.0)
- moved C8 17.5 mm to (109.2, 49.5)
- moved U5 17.5 mm to (112.0, 49.8)
- moved C25 16.2 mm to (112.8, 52.0), turned to 0 degrees
- moved L1 13.8 mm to (118.0, 51.0), turned to 270 degrees
- moved C6 10.2 mm to (119.5, 64.2), turned to 90 degrees
- moved U4 10.2 mm to (116.8, 64.2), turned to 180 degrees
- moved C14 10.0 mm to (118.2, 54.0)
- moved C15 7.04 mm to (119.5, 51.0), turned to 90 degrees
- moved R5 7.04 mm to (121.5, 57.8), turned to 180 degrees
- moved C12 6.62 mm to (118.2, 55.8)
- moved C11 5.50 mm to (139.0, 63.8), turned to 270 degrees
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Routing:
- net +3.3VA: track 0.00 -> 23.2 mm
- net GNDS: track 0.00 -> 17.0 mm
- net +3V3: track 0.00 -> 16.3 mm
- net +5V: track 0.00 -> 15.4 mm
- net 5: track 0.00 -> 13.5 mm, vias 0 -> 1
- net 3: track 0.00 -> 13.4 mm, vias 0 -> 1
- net 1: track 0.00 -> 13.4 mm, vias 0 -> 1
- net 2: track 0.00 -> 11.6 mm, vias 0 -> 1
- net 6: track 0.00 -> 10.8 mm, vias 0 -> 1
- net 4: track 0.00 -> 10.1 mm, vias 0 -> 1
- net Net-(J1-Pad7): track 0.00 -> 9.75 mm
- net Net-(J4-Pad3): track 0.00 -> 9.16 mm
- net Net-(J2-Pad3): track 0.00 -> 9.16 mm
- net Net-(J5-Pad3): track 0.00 -> 8.16 mm
- net Net-(J3-Pad3): track 0.00 -> 8.16 mm
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- added copper zone on F.Cu, net GND

Commit message: hw
Parts:
- moved C6 8.62 mm to (117.0, 56.0), turned to 180 degrees
- moved JP2 8.49 mm to (119.5, 57.0), turned to 90 degrees
- moved JP4 8.49 mm to (119.5, 67.5), turned to 90 degrees
- moved U4 4.50 mm to (116.8, 59.8), turned to 0 degrees
- moved C12 2.85 mm to (116.5, 53.5), turned to 270 degrees
- moved R10 1.50 mm to (120.2, 59.2)
- moved R14 1.50 mm to (133.5, 60.8)
- moved R15 1.50 mm to (133.5, 62.2)
- moved R4 1.50 mm to (120.2, 48.8)
- moved R8 1.50 mm to (133.5, 50.2)
- moved R9 1.50 mm to (133.5, 51.8)
- moved C17 1.25 mm to (123.0, 48.8), turned to 0 degrees
- moved C22 1.25 mm to (123.0, 59.2), turned to 0 degrees
- moved JP1 1.25 mm to (125.8, 48.8)
- moved JP3 1.25 mm to (125.8, 59.2)
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Connections:
- C11 pad 1: +3V3 -> +3.3VA
- C13 pad 1: +3V3 -> +3.3VA
- R2 pad 2: +3V3 -> +5V
- U12 pad 1: Net-(J3-Pad2) -> Net-(J3-Pad3)
- U12 pad 2: B1+ -> B1-
- U12 pad 3: B1- -> B1+
- U12 pad 4: Net-(J3-Pad3) -> Net-(J3-Pad2)
- U14 pad 1: Net-(J5-Pad2) -> Net-(J5-Pad3)
- U14 pad 2: B2+ -> B2-
- U14 pad 3: B2- -> B2+
- U14 pad 4: Net-(J5-Pad3) -> Net-(J5-Pad2)
- U6 pad 4: B1- -> B1+
- U6 pad 5: +3V3 -> +3.3VA
- U6 pad 6: B1+ -> B1-
- U7 pad 4: B2- -> B2+
- U7 pad 5: +3V3 -> +3.3VA
- U7 pad 6: B2+ -> B2-
Routing:
- net +5V: track 15.4 -> 94.9 mm, vias 0 -> 13
- net +3.3VA: track 23.2 -> 76.0 mm, vias 0 -> 4
- net SCK: track 0.00 -> 44.4 mm, vias 0 -> 6
- net GNDS: track 17.0 -> 59.7 mm
- net XSCK: track 0.00 -> 14.9 mm, vias 0 -> 2
- net DOUT1: track 0.00 -> 14.4 mm, vias 0 -> 2
- net DOUT2: track 0.00 -> 14.2 mm, vias 0 -> 2
- net Net-(JP4-Pad1): track 0.00 -> 9.54 mm, vias 0 -> 2
- net Net-(JP2-Pad1): track 0.00 -> 9.54 mm, vias 0 -> 2
- net Net-(C19-Pad1): track 1.25 -> 5.68 mm
- net +3V3: track 16.3 -> 20.4 mm, vias 0 -> 2
- net Net-(C18-Pad1): track 1.25 -> 5.07 mm
- net A2+: track 1.78 -> 5.44 mm
- net A1+: track 1.78 -> 5.44 mm
- net Net-(C22-Pad2): track 0.00 -> 3.11 mm
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- added copper zone on B.Cu, net GND
- added copper zone on B.Cu, net GNDS
- added copper zone on F.Cu, net GNDS
Other:
- board size 66.8 x 22 mm -> 70 x 22 mm

Commit message: parts
Parts:
- R12, R13, R14, R15, R6, R7, R8, R9: value 100 -> 120
- R16, R3: footprint stmbl:C_0603 -> stmbl:R_0603
- U2, U3: value RS485 -> sp485
Other:
- outline, holes or cut-outs redrawn

Commit message: jlc export
Parts:
- renumbered C1 to C301, C2 to C302, C3 to C303, C4 to C304, C6 to C305, C5 to C306, C7 to C307, C8 to C308, C25 to C309, C11 to C310, C9 to C311, C13 to C312, C10 to C313, C12 to C314, C14 to C315, C15 to C316, C16 to C317, C17 to C318, C18 to C319, C19 to C320, C20 to C321, C21 to C322, C22 to C323, C23 to C324, C24 to C325, J1 to J301, J2 to J302, J3 to J303, J4 to J304, J5 to J305, JP1 to JP301, JP2 to JP302, JP3 to JP303, JP4 to JP304, L1 to L301, R2 to R301, R1 to R302, R3 to R303, R16 to R304, R4 to R305, R5 to R306, R6 to R307, R7 to R308, R8 to R309, R9 to R310, R10 to R311, R11 to R312, R12 to R313, R13 to R314, R14 to R315, R15 to R316, U10 to U301, U1 to U302, U2 to U303, U3 to U304, U4 to U305, U5 to U306, U6 to U307, U7 to U308, U11 to U309, U12 to U310, U13 to U311, U14 to U312, U8 to U313, U9 to U314

Commit message: hx711
Parts:
- moved U305 0.50 mm to (116.8, 59.2)
- moved U301 0.25 mm to (103.0, 49.0)
- turned R304 to 270 degrees
Connections:
- U302 pad 6: 2 -> 1
- U302 pad 7: 1 -> 2
- U303 pad 6: 4 -> 5
- U303 pad 7: 5 -> 4
- U304 pad 6: 6 -> 3
- U304 pad 7: 3 -> 6
Routing:
- net 5: track 13.6 -> 12.4 mm, vias 1 -> 0
- net XSCK: track 14.9 -> 14.0 mm
- net 4: track 10.2 -> 10.9 mm, vias 1 -> 0
- net Net-(J301-Pad8): track 6.75 -> 7.29 mm
- net 3: track 13.4 -> 13.9 mm
- net 6: track 10.8 -> 10.3 mm, vias 1 -> 0
- net 2: track 12.7 -> 13.0 mm, vias 1 -> 0
Other:
- board text added: "STMBL HX711 BOB V1.1"
- board text added: "int. clock"
- board text added: "rate"
