File: hx711/pcb.sch (KiCad schematic (older format))
At the start: 30 parts, among them J1 RJ45_LED, J2 CONN_02X03_Odd_Even, J3 CONN_02X03_Odd_Even, J4 CONN_02X03_Odd_Even, J5 CONN_02X03_Odd_Even, U1 sp485, U2 RS485, U3 RS485, U4 20M, U5 MIC55, U6 USBLC6-4SC6, U7 USBLC6-4SC6

Commit message: hx711
Parts:
- added R16: 120, stmbl:C_0603, symbol stmbl:R
- C1, C10, C11, C13, C14, C2, C3, C4, C6, C8: footprint stmbl:C0603 -> stmbl:C_0603
- C12, C5, C7, C9: footprint stmbl:C0805 -> stmbl:C_0805
- L1: footprint stmbl:R0603 -> stmbl:R_0603
- R1, R2, R3: footprint (none) -> stmbl:C_0603
- U4: footprint (none) -> stmbl:Oscillator_SMD_0603_4Pads
Connections:
- net 4: now also R16.2
- net 5: now also R16.1
- net A1+: now also U6.3 (IO2); no longer U6.1 (IO1)
- net A1-: now also U6.1 (IO1); no longer U6.3 (IO2)
- net A2+: now also U7.3 (IO2); no longer U7.1 (IO1)
- net A2-: now also U7.1 (IO1); no longer U7.3 (IO2)
Changed lines of the file:
@@
 EESchema Schematic File Version 4
+LIBS:pcb-cache
 EELAYER 30 0
 EELAYER END
@@
 F 0 "C2" V 4102 1900 50  0000 C CNN
 F 1 "100n" V 4011 1900 50  0000 C CNN
-F 2 "stmbl:C0603" H 3965 1809 50  0001 L CNN
+F 2 "stmbl:C_0603" H 3965 1809 50  0001 L CNN
 F 3 "" H 3850 1900 50  0001 C CNN
 	1    3850 1900
@@
 F 0 "U4" H 6200 1397 60  0000 C CNN
 F 1 "20M" H 6200 1291 60  0000 C CNN
-F 2 "" H 6200 1100 60  0001 C CNN
+F 2 "stmbl:Oscillator_SMD_0603_4Pads" H 6200 1100 60  0001 C CNN
 F 3 "" H 6200 1100 60  0001 C CNN
 F 4 "Q33310F70051500" H 6200 1100 50  0001 C CNN "Manufacturer No"
@@
 F 0 "L1" V 7666 5250 50  0000 C CNN
 F 1 "INDUCTOR" V 7575 5250 50  0000 C CNN
-F 2 "stmbl:R0603" V 7575 5250 50  0001 C CNN
+F 2 "stmbl:R_0603" V 7575 5250 50  0001 C CNN
 F 3 "" H 7450 5250 50  0001 C CNN
 	1    7450 5250
@@
 F 0 "C9" H 6815 5546 50  0000 L CNN
 F 1 "10u" H 6815 5455 50  0000 L CNN
-F 2 "stmbl:C0805" H 6815 5409 50  0001 L CNN
+F 2 "stmbl:C_0805" H 6815 5409 50  0001 L CNN
 F 3 "" H 6700 5500 50  0001 C CNN
 	1    6700 5500
@@
 F 0 "C10" H 7165 5546 50  0000 L CNN
 F 1 "100n" H 7165 5455 50  0000 L CNN
-F 2 "stmbl:C0603" H 7165 5409 50  0001 L CNN
+F 2 "stmbl:C_0603" H 7165 5409 50  0001 L CNN
 F 3 "" H 7050 5500 50  0001 C CNN
 	1    7050 5500
@@
 F 0 "C8" H 5665 5546 50  0000 L CNN
 F 1 "100n" H 5665 5455 50  0000 L CNN
-F 2 "stmbl:C0603" H 5665 5409 50  0001 L CNN
+F 2 "stmbl:C_0603" H 5665 5409 50  0001 L CNN
 F 3 "" H 5550 5500 50  0001 C CNN
 	1    5550 5500
@@
 F 0 "C7" H 5315 5546 50  0000 L CNN
 F 1 "10u" H 5315 5455 50  0000 L CNN
-F 2 "stmbl:C0805" H 5315 5409 50  0001 L CNN
+F 2 "stmbl:C_0805" H 5315 5409 50  0001 L CNN
 F 3 "" H 5200 5500 50  0001 C CNN
 	1    5200 5500
@@
 F 0 "C12" H 7965 5546 50  0000 L CNN
 F 1 "10u" H 7965 5455 50  0000 L CNN
-F 2 "stmbl:C0805" H 7965 5409 50  0001 L CNN
+F 2 "stmbl:C_0805" H 7965 5409 50  0001 L CNN
 F 3 "" H 7850 5500 50  0001 C CNN
 	1    7850 5500
@@
 F 0 "C6" H 5265 1146 50  0000 L CNN
 F 1 "100n" H 5265 1055 50  0000 L CNN
-F 2 "stmbl:C0603" H 5265 1009 50  0001 L CNN
+F 2 "stmbl:C_0603" H 5265 1009 50  0001 L CNN
 F 3 "" H 5150 1100 50  0001 C CNN
 	1    5150 1100
@@
 F 0 "C11" H 7765 1246 50  0000 L CNN
 F 1 "100n" H 7765 1155 50  0000 L CNN
-F 2 "stmbl:C0603" H 7765 1109 50  0001 L CNN
+F 2 "stmbl:C_0603" H 7765 1109 50  0001 L CNN
 F 3 "" H 7650 1200 50  0001 C CNN
 	1    7650 1200
@@
 F 0 "C13" H 8165 1246 50  0000 L CNN
 F 1 "100n" H 8165 1155 50  0000 L CNN
-F 2 "stmbl:C0603" H 8165 1109 50  0001 L CNN
+F 2 "stmbl:C_0603" H 8165 1109 50  0001 L CNN
 F 3 "" H 8050 1200 50  0001 C CNN
 	1    8050 1200
@@
 	5600 2150 5700 2150
 Text GLabel 5600 3150 0    60   Input ~ 0
-DOUT1
+DOUT2
 Wire Wire Line
 	5600 3150 5700 3150
@@
 Wire Wire Line
 	8450 2000 8350 2000
+Text GLabel 7250 2400 0    60   Input ~ 0
+A1+
 Text GLabel 7250 2000 0    60   Input ~ 0
-A1+
-Text GLabel 7250 2400 0    60   Input ~ 0
 A1-
 Text GLabel 8450 2000 2    60   Input ~ 0
@@
 Wire Wire Line
 	8450 3000 8350 3000
+Text GLabel 7250 3400 0    60   Input ~ 0
+A2+
 Text GLabel 7250 3000 0    60   Input ~ 0
-A2+
-Text GLabel 7250 3400 0    60   Input ~ 0
 A2-
 Text GLabel 8450 3000 2    60   Input ~ 0
@@
 F 0 "C3" V 4102 2850 50  0000 C CNN
 F 1 "100n" V 4011 2850 50  0000 C CNN
-F 2 "stmbl:C0603" H 3965 2759 50  0001 L CNN
+F 2 "stmbl:C_0603" H 3965 2759 50  0001 L CNN
 F 3 "" H 3850 2850 50  0001 C CNN
 	1    3850 2850
@@
 F 0 "C4" V 4102 3800 50  0000 C CNN
 F 1 "100n" V 4011 3800 50  0000 C CNN
-F 2 "stmbl:C0603" H 3965 3709 50  0001 L CNN
+F 2 "stmbl:C_0603" H 3965 3709 50  0001 L CNN
 F 3 "" H 3850 3800 50  0001 C CNN
 	1    3850 3800
@@
 F 0 "C1" H 2265 3796 50  0000 L CNN
 F 1 "100n" H 2265 3705 50  0000 L CNN
-F 2 "stmbl:C0603" H 2265 3659 50  0001 L CNN
+F 2 "stmbl:C_0603" H 2265 3659 50  0001 L CNN
 F 3 "" H 2150 3750 50  0001 C CNN
 	1    2150 3750
@@
 F 0 "R3" H 1920 3796 50  0000 L CNN
 F 1 "120" H 1920 3705 50  0000 L CNN
-F 2 "" V 1780 3750 50  0001 C CNN
+F 2 "stmbl:C_0603" V 1780 3750 50  0001 C CNN
 F 3 "" H 1850 3750 50  0001 C CNN
 	1    1850 3750
@@
 F 0 "C14" H 8315 5546 50  0000 L CNN
 F 1 "2.2u" H 8315 5455 50  0000 L CNN
-F 2 "stmbl:C0603" H 8315 5409 50  0001 L CNN
+F 2 "stmbl:C_0603" H 8315 5409 50  0001 L CNN
 F 3 "" H 8200 5500 50  0001 C CNN
 	1    8200 5500
@@
 F 0 "R1" V 993 3050 50  0000 C CNN
 F 1 "560" V 1084 3050 50  0000 C CNN
-F 2 "" V 1130 3050 50  0001 C CNN
+F 2 "stmbl:C_0603" V 1130 3050 50  0001 C CNN
 F 3 "" H 1200 3050 50  0001 C CNN
 	1    1200 3050
@@
 F 0 "R2" V 1043 2350 50  0000 C CNN
 F 1 "560" V 1134 2350 50  0000 C CNN
-F 2 "" V 1180 2350 50  0001 C CNN
+F 2 "stmbl:C_0603" V 1180 2350 50  0001 C CNN
 F 3 "" H 1250 2350 50  0001 C CNN
 	1    1250 2350
@@
 F 0 "C5" H 4965 5546 50  0000 L CNN
 F 1 "10u" H 4965 5455 50  0000 L CNN
-F 2 "stmbl:C0805" H 4965 5409 50  0001 L CNN
+F 2 "stmbl:C_0805" H 4965 5409 50  0001 L CNN
 F 3 "" H 4850 5500 50  0001 C CNN
 	1    4850 5500
@@
 	1    0    0    -1
 $EndComp
+$Comp
+L stmbl:R R16
+U 1 1 5E2A356F
+P 3000 3350
+F 0 "R16" H 3070 3396 50  0000 L CNN
+F 1 "120" H 3070 3305 50  0000 L CNN
+F 2 "stmbl:C_0603" V 2930 3350 50  0001 C CNN
+F 3 "" H 3000 3350 50  0001 C CNN
+	1    3000 3350
+	1    0    0    -1
+$EndComp
+Text GLabel 3000 3100 1    60   Input ~ 0
+5
+Wire Wire Line
+	3000 3100 3000 3200
+Text GLabel 3000 3600 3    60   Input ~ 0
+4
+Wire Wire Line
+	3000 3600 3000 3500
 $EndSCHEMATC

Commit message: hx711
Parts:
- removed J2, J3, J4, J5: CONN_02X03_Odd_Even, stmbl:Pin_Header_RM2.54_2x3_UP, symbol stmbl:CONN_02X03_Odd_Even
- removed U5: MIC55, stmbl:SOT-23-5, symbol stmbl:MIC55
- added C25: 100p, stmbl:C_0603, symbol stmbl:C
- added J2, J3, J4, J5: CONN_01X05, stmbl:Pin_Header_RM2.54_1x5_UP, symbol stmbl:CONN_01X05
- added U10, U11, U12, U13, U14: CMC, stmbl:CMC_0805, symbol stmbl:CMC
- added U5: LDO, stmbl:SOT-23-5, symbol stmbl:LDO
Connections:
- net +3.3VA: now also J2.1 (Pin_1), J3.1 (Pin_1), J4.1 (Pin_1), J5.1 (Pin_1)
- net +3V3: now also U5.5 (VOUT)
- net +5V: now also U10.3, U5.1 (VIN), U5.3 (EN); no longer J1.7
- net A1+: now also U11.2
- net A1-: now also U11.3
- net A2+: now also U13.2
- net A2-: now also U13.3
- net B1+: now also U12.2
- net B1-: now also U12.3
- net B2+: now also U14.2
- net B2-: now also U14.3
- net GND: now also C25.1, J2.4 (Pin_4), J3.4 (Pin_4), J4.4 (Pin_4), J5.4 (Pin_4), U10.2, U5.2 (GND); no longer J1.8
- net GNDS: now also J2.5 (Pin_5), J3.5 (Pin_5), J4.5 (Pin_5), J5.5 (Pin_5)
- net SCK: now also U2.1 (RO); no longer U2.4 (DI)
- new net: J2.2 (Pin_2), U11.1
- new net: J2.3 (Pin_3), U11.4
- new net: J1.7, U10.4
- new net: J1.8, U10.1
- new net: J3.2 (Pin_2), U12.1
- new net: J3.3 (Pin_3), U12.4
- new net: J4.2 (Pin_2), U13.1
- new net: J4.3 (Pin_3), U13.4
- new net: J5.2 (Pin_2), U14.1
- new net: J5.3 (Pin_3), U14.4
- new net: C25.2, U5.4 (BYP)
Other:
- moved on the sheet: C1, C10, C11, C12, C13, C14, C2, C3, C4, C5, C6, C7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

Commit message: hw
Connections:
- net +3.3VA: now also C11.1, C13.1, U6.5 (VBUS), U7.5 (VBUS)
- net +3V3: no longer C11.1, C13.1, R2.2, U6.5 (VBUS), U7.5 (VBUS)
- net +5V: now also R2.2
- net B1+: now also U12.3, U6.4 (IO3); no longer U12.2, U6.6 (IO4)
- net B1-: now also U12.2, U6.6 (IO4); no longer U12.3, U6.4 (IO3)
- net B2+: now also U14.3, U7.4 (IO3); no longer U14.2, U7.6 (IO4)
- net B2-: now also U14.2, U7.6 (IO4); no longer U14.3, U7.4 (IO3)
- net at U12.1: now also J3.3 (Pin_3); no longer J3.2 (Pin_2)
- net at U12.4: now also J3.2 (Pin_2); no longer J3.3 (Pin_3)
- net at U14.1: now also J5.3 (Pin_3); no longer J5.2 (Pin_2)
- net at U14.4: now also J5.2 (Pin_2); no longer J5.3 (Pin_3)
Changed lines of the file:
@@
 	8550 3250 8450 3250
-$Comp
-L stmbl:+3.3V #PWR039
-U 1 1 5E451397
-P 8550 3250
-F 0 "#PWR039" H 8550 3100 50  0001 C CNN
-F 1 "+3.3V" V 8565 3378 50  0000 L CNN
-F 2 "" H 8550 3250 50  0001 C CNN
-F 3 "" H 8550 3250 50  0001 C CNN
-	1    8550 3250
-	0    1    1    0
-$EndComp
-$Comp
-L stmbl:+3.3V #PWR038
-U 1 1 5E451F3C
-P 8550 2250
-F 0 "#PWR038" H 8550 2100 50  0001 C CNN
-F 1 "+3.3V" V 8565 2378 50  0000 L CNN
-F 2 "" H 8550 2250 50  0001 C CNN
-F 3 "" H 8550 2250 50  0001 C CNN
-	1    8550 2250
-	0    1    1    0
-$EndComp
-$Comp
-L stmbl:+3.3V #PWR036
-U 1 1 5E4524EB
-P 8150 1000
-F 0 "#PWR036" H 8150 850 50  0001 C CNN
-F 1 "+3.3V" H 8165 1173 50  0000 C CNN
-F 2 "" H 8150 1000 50  0001 C CNN
-F 3 "" H 8150 1000 50  0001 C CNN
-	1    8150 1000
-	1    0    0    -1
-$EndComp
-$Comp
-L stmbl:+3.3V #PWR033
-U 1 1 5E452F59
-P 7750 1000
-F 0 "#PWR033" H 7750 850 50  0001 C CNN
-F 1 "+3.3V" H 7765 1173 50  0000 C CNN
-F 2 "" H 7750 1000 50  0001 C CNN
-F 3 "" H 7750 1000 50  0001 C CNN
-	1    7750 1000
-	1    0    0    -1
-$EndComp
 $Comp
 L stmbl:GND #PWR034
@@
 Text GLabel 7350 2050 0    60   Input ~ 0
 A1-
+Text GLabel 8550 2450 2    60   Input ~ 0
+B1+
 Text GLabel 8550 2050 2    60   Input ~ 0
-B1+
-Text GLabel 8550 2450 2    60   Input ~ 0
 B1-
 Wire Wire Line
@@
 Text GLabel 7350 3050 0    60   Input ~ 0
 A2-
+Text GLabel 8550 3450 2    60   Input ~ 0
+B2+
 Text GLabel 8550 3050 2    60   Input ~ 0
-B2+
-Text GLabel 8550 3450 2    60   Input ~ 0
 B2-
 $Comp
@@
 Connection ~ 8950 5550
 $Comp
-L stmbl:+3.3V #PWR01
-U 1 1 5E5D9FF4
-P 900 2150
-F 0 "#PWR01" H 900 2000 50  0001 C CNN
-F 1 "+3.3V" V 915 2278 50  0000 L CNN
-F 2 "" H 900 2150 50  0001 C CNN
-F 3 "" H 900 2150 50  0001 C CNN
-	1    900  2150
-	0    -1   -1   0
-$EndComp
-$Comp
 L stmbl:R R16
 U 1 1 5E2A356F
@@
 F 4 "DLW21HN900SQ2L" H 9800 2500 50  0001 C CNN "Manufacturer No"
 	1    9800 2500
-	-1   0    0    -1
+	-1   0    0    1
 $EndComp
 $Comp
@@
 F 4 "DLW21HN900SQ2L" H 9800 3800 50  0001 C CNN "Manufacturer No"
 	1    9800 3800
-	-1   0    0    -1
+	-1   0    0    1
 $EndComp
 $Comp
@@
 Connection ~ 7600 5550
 Connection ~ 7800 5550
+$Comp
+L stmbl:+3.3VA #PWR0113
+U 1 1 5E8F2936
+P 8550 2250
+F 0 "#PWR0113" H 8550 2100 50  0001 C CNN
+F 1 "+3.3VA" V 8565 2377 50  0000 L CNN
+F 2 "" H 8550 2250 50  0001 C CNN
+F 3 "" H 8550 2250 50  0001 C CNN
+	1    8550 2250
+	0    1    1    0
+$EndComp
+$Comp
+L stmbl:+3.3VA #PWR0114
+U 1 1 5E8F3130
+P 8550 3250
+F 0 "#PWR0114" H 8550 3100 50  0001 C CNN
+F 1 "+3.3VA" V 8565 3377 50  0000 L CNN
+F 2 "" H 8550 3250 50  0001 C CNN
+F 3 "" H 8550 3250 50  0001 C CNN
+	1    8550 3250
+	0    1    1    0
+$EndComp
+$Comp
+L stmbl:+3.3VA #PWR0115
+U 1 1 5E8F439C
+P 8150 1000
+F 0 "#PWR0115" H 8150 850 50  0001 C CNN
+F 1 "+3.3VA" V 8165 1127 50  0000 L CNN
+F 2 "" H 8150 1000 50  0001 C CNN
+F 3 "" H 8150 1000 50  0001 C CNN
+	1    8150 1000
+	1    0    0    -1
+$EndComp
+$Comp
+L stmbl:+3.3VA #PWR0116
+U 1 1 5E8F4B61
+P 7750 1000
+F 0 "#PWR0116" H 7750 850 50  0001 C CNN
+F 1 "+3.3VA" V 7765 1127 50  0000 L CNN
+F 2 "" H 7750 1000 50  0001 C CNN
+F 3 "" H 7750 1000 50  0001 C CNN
+	1    7750 1000
+	1    0    0    -1
+$EndComp
+$Comp
+L stmbl:+5V #PWR?
+U 1 1 5E8F5667
+P 900 2150
+F 0 "#PWR?" H 900 2000 50  0001 C CNN
+F 1 "+5V" V 915 2278 50  0000 L CNN
+F 2 "" H 900 2150 50  0001 C CNN
+F 3 "" H 900 2150 50  0001 C CNN
+	1    900  2150
+	0    -1   -1   0
+$EndComp
 $EndSCHEMATC

Commit message: parts
Parts:
- C1, C10, C11, C13, C2, C3, C4, C6, C8: LCSC (none) -> C14663
- C12, C5, C7, C9: LCSC (none) -> C15850
- C14: LCSC (none) -> C23630
- C25: LCSC (none) -> C14858
- L1: LCSC (none) -> C73100
- R1, R2: LCSC (none) -> C23204
- R16, R3: footprint stmbl:C_0603 -> stmbl:R_0603; LCSC (none) -> C22787
- U1: LCSC (none) -> C6855
- U10, U11, U12, U13, U14: LCSC (none) -> C80529
- U2, U3: value RS485 -> sp485; LCSC (none) -> C6855
- U4: LCSC (none) -> C32529
- U5: LCSC (none) -> C9055
- U6, U7: LCSC (none) -> C111212
Changed lines of the file:
@@
 F 2 "stmbl:C_0603" H 4515 1609 50  0001 L CNN
 F 3 "" H 4400 1700 50  0001 C CNN
+F 4 "C14663" H 4400 1700 50  0001 C CNN "LCSC"
 	1    4400 1700
 	0    -1   -1   0
@@
 F 2 "stmbl:SOIC-8-N" H 4400 2483 50  0001 C CIN
 F 3 "" H 4400 2200 50  0001 C CNN
+F 4 "C6855" H 4400 2200 50  0001 C CNN "LCSC"
 	1    4400 2200
 	-1   0    0    -1
@@
 F 3 "" H 6300 1150 60  0001 C CNN
 F 4 "Q33310F70051500" H 6300 1150 50  0001 C CNN "Manufacturer No"
+F 5 "C32529" H 6300 1150 50  0001 C CNN "LCSC"
 	1    6300 1150
 	1    0    0    -1
@@
 F 2 "stmbl:R_0603" V 8675 5050 50  0001 C CNN
 F 3 "" H 8550 5050 50  0001 C CNN
+F 4 "C73100" H 8550 5050 50  0001 C CNN "LCSC"
 	1    8550 5050
 	0    -1   -1   0
@@
 F 2 "stmbl:C_0805" H 7915 5209 50  0001 L CNN
 F 3 "" H 7800 5300 50  0001 C CNN
+F 4 "C15850" H 7800 5300 50  0001 C CNN "LCSC"
 	1    7800 5300
 	1    0    0    -1
@@
 F 2 "stmbl:C_0603" H 8265 5209 50  0001 L CNN
 F 3 "" H 8150 5300 50  0001 C CNN
+F 4 "C14663" H 8150 5300 50  0001 C CNN "LCSC"
 	1    8150 5300
 	1    0    0    -1
@@
 F 2 "stmbl:C_0603" H 6115 5209 50  0001 L CNN
 F 3 "" H 6000 5300 50  0001 C CNN
+F 4 "C14663" H 6000 5300 50  0001 C CNN "LCSC"
 	1    6000 5300
 	1    0    0    -1
@@
 F 2 "stmbl:C_0805" H 5765 5209 50  0001 L CNN
 F 3 "" H 5650 5300 50  0001 C CNN
+F 4 "C15850" H 5650 5300 50  0001 C CNN "LCSC"
 	1    5650 5300
 	1    0    0    -1
@@
 F 2 "stmbl:C_0805" H 9065 5209 50  0001 L CNN
 F 3 "" H 8950 5300 50  0001 C CNN
+F 4 "C15850" H 8950 5300 50  0001 C CNN "LCSC"
 	1    8950 5300
 	1    0    0    -1
@@
 F 2 "stmbl:C_0603" H 5365 1059 50  0001 L CNN
 F 3 "" H 5250 1150 50  0001 C CNN
+F 4 "C14663" H 5250 1150 50  0001 C CNN "LCSC"
 	1    5250 1150
 	1    0    0    -1
@@
 F 2 "stmbl:SOT-23-6" H 8250 2700 50  0001 C CNN
 F 3 "" H 7700 2600 50  0001 C CNN
+F 4 "C111212" H 7950 2250 50  0001 C CNN "LCSC"
 	1    7950 2250
 	1    0    0    -1
@@
 F 2 "stmbl:SOT-23-6" H 8250 3700 50  0001 C CNN
 F 3 "" H 7700 3600 50  0001 C CNN
+F 4 "C111212" H 7950 3250 50  0001 C CNN "LCSC"
 	1    7950 3250
 	1    0    0    -1
@@
 F 2 "stmbl:C_0603" H 7865 1159 50  0001 L CNN
 F 3 "" H 7750 1250 50  0001 C CNN
+F 4 "C14663" H 7750 1250 50  0001 C CNN "LCSC"
 	1    7750 1250
 	1    0    0    -1
@@
 F 2 "stmbl:C_0603" H 8265 1159 50  0001 L CNN
 F 3 "" H 8150 1250 50  0001 C CNN
+F 4 "C14663" H 8150 1250 50  0001 C CNN "LCSC"
 	1    8150 1250
 	1    0    0    -1
@@
 F 2 "stmbl:C_0603" H 4515 2559 50  0001 L CNN
 F 3 "" H 4400 2650 50  0001 C CNN
+F 4 "C14663" H 4400 2650 50  0001 C CNN "LCSC"
 	1    4400 2650
 	0    -1   -1   0
@@
 P 4400 3150
 F 0 "U2" H 4400 3525 50  0000 C CNN
-F 1 "RS485" H 4400 3434 50  0000 C CNN
+F 1 "sp485" H 4400 3434 50  0000 C CNN
 F 2 "stmbl:SOIC-8-N" H 4400 3433 50  0001 C CIN
 F 3 "" H 4400 3150 50  0001 C CNN
+F 4 "C6855" H 4400 3150 50  0001 C CNN "LCSC"
 	1    4400 3150
 	-1   0    0    -1
@@
 F 2 "stmbl:C_0603" H 4515 3509 50  0001 L CNN
 F 3 "" H 4400 3600 50  0001 C CNN
+F 4 "C14663" H 4400 3600 50  0001 C CNN "LCSC"
 	1    4400 3600
 	0    -1   -1   0
@@
 P 4400 4100
 F 0 "U3" H 4400 4475 50  0000 C CNN
-F 1 "RS485" H 4400 4384 50  0000 C CNN
+F 1 "sp485" H 4400 4384 50  0000 C CNN
 F 2 "stmbl:SOIC-8-N" H 4400 4383 50  0001 C CIN
 F 3 "" H 4400 4100 50  0001 C CNN
+F 4 "C6855" H 4400 4100 50  0001 C CNN "LCSC"
 	1    4400 4100
 	-1   0    0    -1
@@
 F 2 "stmbl:C_0603" H 2165 3459 50  0001 L CNN
 F 3 "" H 2050 3550 50  0001 C CNN
+F 4 "C14663" H 2050 3550 50  0001 C CNN "LCSC"
 	1    2050 3550
 	1    0    0    -1
@@
 F 0 "R3" H 1820 3596 50  0000 L CNN
 F 1 "120" H 1820 3505 50  0000 L CNN
-F 2 "stmbl:C_0603" V 1680 3550 50  0001 C CNN
+F 2 "stmbl:R_0603" V 1680 3550 50  0001 C CNN
 F 3 "" H 1750 3550 50  0001 C CNN
+F 4 "C22787" H 1750 3550 50  0001 C CNN "LCSC"
 	1    1750 3550
 	1    0    0    -1
@@
 F 2 "stmbl:C_0603" H 9415 5209 50  0001 L CNN
 F 3 "" H 9300 5300 50  0001 C CNN
+F 4 "C23630" H 9300 5300 50  0001 C CNN "LCSC"
 	1    9300 5300
 	1    0    0    -1
@@
 F 2 "stmbl:C_0603" V 1080 2850 50  0001 C CNN
 F 3 "" H 1150 2850 50  0001 C CNN
+F 4 "C23204" H 1150 2850 50  0001 C CNN "LCSC"
 	1    1150 2850
 	0    1    1    0
@@
 F 2 "stmbl:C_0603" V 1080 2150 50  0001 C CNN
 F 3 "" H 1150 2150 50  0001 C CNN
+F 4 "C23204" H 1150 2150 50  0001 C CNN "LCSC"
 	1    1150 2150
 	0    1    1    0
@@
 F 2 "stmbl:C_0805" H 5415 5209 50  0001 L CNN
 F 3 "" H 5300 5300 50  0001 C CNN
+F 4 "C15850" H 5300 5300 50  0001 C CNN "LCSC"
 	1    5300 5300
 	1    0    0    -1
@@
 F 0 "R16" H 3620 3196 50  0000 L CNN
 F 1 "120" H 3620 3105 50  0000 L CNN
-F 2 "stmbl:C_0603" V 3480 3150 50  0001 C CNN
+F 2 "stmbl:R_0603" V 3480 3150 50  0001 C CNN
 F 3 "" H 3550 3150 50  0001 C CNN
+F 4 "C22787" H 3550 3150 50  0001 C CNN "LCSC"
 	1    3550 3150
 	1    0    0    -1
@@
 F 3 "" H 9800 1850 60  0001 C CNN
 F 4 "DLW21HN900SQ2L" H 9800 1850 50  0001 C CNN "Manufacturer No"
+F 5 "C80529" H 9800 1850 50  0001 C CNN "LCSC"
 	1    9800 1850
 	-1   0    0    -1
@@
 F 3 "" H 9800 2500 60  0001 C CNN
 F 4 "DLW21HN900SQ2L" H 9800 2500 50  0001 C CNN "Manufacturer No"
+F 5 "C80529" H 9800 2500 50  0001 C CNN "LCSC"
 	1    9800 2500
 	-1   0    0    1
@@
 F 3 "" H 9800 3150 60  0001 C CNN
 F 4 "DLW21HN900SQ2L" H 9800 3150 50  0001 C CNN "Manufacturer No"
+F 5 "C80529" H 9800 3150 50  0001 C CNN "LCSC"
 	1    9800 3150
 	-1   0    0    -1
@@
 F 3 "" H 9800 3800 60  0001 C CNN
 F 4 "DLW21HN900SQ2L" H 9800 3800 50  0001 C CNN "Manufacturer No"
+F 5 "C80529" H 9800 3800 50  0001 C CNN "LCSC"
 	1    9800 3800
 	-1   0    0    1
@@
 F 3 "" H 2700 2900 60  0001 C CNN
 F 4 "DLW21HN900SQ2L" H 2700 2900 50  0001 C CNN "Manufacturer No"
+F 5 "C80529" H 2700 2900 50  0001 C CNN "LCSC"
 	1    2700 2900
 	1    0    0    1
@@
 F 3 "" H 6750 5150 50  0000 C CNN
 F 4 "AP2202K-3.3TRG1" H 6750 5150 50  0001 C CNN "Manufacturer No"
+F 5 "C9055" H 6750 5150 50  0001 C CNN "LCSC"
 	1    6750 5150
 	1    0    0    -1
@@
 F 2 "stmbl:C_0603" H 7465 5159 50  0001 L CNN
 F 3 "" H 7350 5250 50  0001 C CNN
+F 4 "C14858" H 7350 5250 50  0001 C CNN "LCSC"
 	1    7350 5250
 	0    1    1    0

Commit message: jlc export
Parts:
- renumbered C1 to C301, C2 to C302, C3 to C303, C4 to C304, C6 to C305, C5 to C306, C7 to C307, C8 to C308, C25 to C309, C11 to C310, C9 to C311, C13 to C312, C10 to C313, C12 to C314, C14 to C315, J1 to J301, J2 to J302, J3 to J303, J4 to J304, J5 to J305, L1 to L301, R2 to R301, R1 to R302, R3 to R303, R16 to R304, U10 to U301, U1 to U302, U2 to U303, U3 to U304, U4 to U305, U5 to U306, U6 to U307, U7 to U308, U11 to U309, U12 to U310, U13 to U311, U14 to U312

Commit message: hx711
Connections:
- net 1: now also U302.6 (A); no longer U302.7 (B)
- net 2: now also U302.7 (B); no longer U302.6 (A)
- net 3: now also U304.6 (A); no longer U304.7 (B)
- net 4: now also U303.7 (B); no longer U303.6 (A)
- net 5: now also U303.6 (A); no longer U303.7 (B)
- net 6: now also U304.7 (B); no longer U304.6 (A)
Changed lines of the file:
@@
 	0    1    1    0
 $EndComp
+Text GLabel 3950 2250 0    60   Input ~ 0
+1
 Text GLabel 3950 2150 0    60   Input ~ 0
-1
-Text GLabel 3950 2250 0    60   Input ~ 0
 2
 Text GLabel 4850 2350 2    60   Input ~ 0
@@
 Wire Wire Line
 	3950 3100 4050 3100
+Text GLabel 3950 3200 0    60   Input ~ 0
+5
 Text GLabel 3950 3100 0    60   Input ~ 0
-5
-Text GLabel 3950 3200 0    60   Input ~ 0
 4
 Text GLabel 4850 3000 2    60   Input ~ 0
@@
 Wire Wire Line
 	3950 4050 4050 4050
+Text GLabel 3950 4150 0    60   Input ~ 0
+3
 Text GLabel 3950 4050 0    60   Input ~ 0
-3
-Text GLabel 3950 4150 0    60   Input ~ 0
 6
 Text GLabel 4850 4250 2    60   Input ~ 0
