File: rs485/pcb.kicad_pcb (KiCad board)
At the start: 4 copper layers, 66.8 x 22 mm, 33 parts, among them J1 RJ45_LED, J2 CONN_02X06_Odd_Even, U1 LDO, U2 sp485, U3 sp485, U4 sp485

Commit message: hw
Parts:
- moved R2 1.50 mm to (105.2, 62.2), turned to 90 degrees
- moved C1 0.25 mm to (103.2, 67.8)
- moved C3 0.25 mm to (108.8, 50.0)
- moved C4 0.25 mm to (114.8, 51.2)
- moved C5 0.25 mm to (114.8, 49.2)
- moved C6 0.25 mm to (117.0, 50.2)
- moved C7 0.25 mm to (106.0, 67.8)
- moved C8 0.25 mm to (106.8, 63.0)
- moved C9 0.25 mm to (106.8, 57.5)
- moved JP1 0.25 mm to (116.5, 68.0)
- moved JP2 0.25 mm to (116.5, 62.5)
- moved JP3 0.25 mm to (116.5, 57.0)
- moved R10 0.25 mm to (106.8, 65.8)
- moved R11 0.25 mm to (116.5, 65.2)
- moved R12 0.25 mm to (106.8, 60.2)
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Connections:
- R2 pad 2: +3V3 -> +5V
Routing:
- net +5V: track 0.00 -> 102.3 mm, vias 0 -> 9
- net GNDS: track 0.00 -> 48.1 mm
- net +3V3: track 0.00 -> 30.2 mm
- net LED: track 0.00 -> 26.8 mm, vias 0 -> 1
- net 1: track 0.00 -> 13.7 mm
- net 4: track 0.00 -> 13.3 mm, vias 0 -> 1
- net 5: track 0.00 -> 13.1 mm, vias 0 -> 1
- net Net-(J2-Pad5): track 0.00 -> 12.7 mm
- net 3: track 0.00 -> 12.3 mm
- net 2: track 0.00 -> 12.0 mm
- net Net-(J2-Pad7): track 0.00 -> 11.4 mm
- net Net-(J2-Pad9): track 0.00 -> 11.2 mm
- net 6: track 0.00 -> 11.1 mm
- net Net-(J2-Pad6): track 0.00 -> 10.4 mm
- net Net-(J2-Pad8): track 0.00 -> 9.21 mm
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- added copper zone on B.Cu, net GND

Commit message: parts
Other:
- board size 66.8 x 22 mm -> 51.8 x 22 mm
Changed lines of the file:
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@@
   (general
     (thickness 1.6)
-    (drawings 14)
+    (drawings 18)
     (tracks 205)
     (zones 0)
@@
     )
   )
-  (gr_arc (start 135 52.5) (end 135 51.5) (angle -180) (layer Edge.Cuts) (width 0.15))
-  (gr_line (start 135 51.5) (end 137.5 51.5) (layer Edge.Cuts) (width 0.15))
-  (gr_arc (start 137.5 52.5) (end 137.5 53.5) (angle -180) (layer Edge.Cuts) (width 0.15))
-  (gr_line (start 135 53.5) (end 137.5 53.5) (layer Edge.Cuts) (width 0.15))
-  (gr_line (start 135 66.25) (end 137.5 66.25) (layer Edge.Cuts) (width 0.15))
-  (gr_line (start 135 64.25) (end 137.5 64.25) (layer Edge.Cuts) (width 0.15))
-  (gr_arc (start 137.5 65.25) (end 137.5 66.25) (angle -180) (layer Edge.Cuts) (width 0.15))
-  (gr_arc (start 135 65.25) (end 135 64.25) (angle -180) (layer Edge.Cuts) (width 0.15))
+  (gr_arc (start 141.5 68.5) (end 141.5 69.5) (angle -90) (layer Edge.Cuts) (width 0.15))
+  (gr_arc (start 91.75 68.5) (end 90.75 68.5) (angle -90) (layer Edge.Cuts) (width 0.15))
+  (gr_arc (start 91.75 48.5) (end 91.75 47.5) (angle -90) (layer Edge.Cuts) (width 0.15))
+  (gr_arc (start 141.5 48.5) (end 142.5 48.5) (angle -90) (layer Edge.Cuts) (width 0.15))
+  (gr_arc (start 136.5 52.5) (end 136.5 51.5) (angle -180) (layer Edge.Cuts) (width 0.15))
+  (gr_line (start 136.5 51.5) (end 139 51.5) (layer Edge.Cuts) (width 0.15))
+  (gr_arc (start 139 52.5) (end 139 53.5) (angle -180) (layer Edge.Cuts) (width 0.15))
+  (gr_line (start 136.5 53.5) (end 139 53.5) (layer Edge.Cuts) (width 0.15))
+  (gr_line (start 136.5 66.25) (end 139 66.25) (layer Edge.Cuts) (width 0.15))
+  (gr_line (start 136.5 64.25) (end 139 64.25) (layer Edge.Cuts) (width 0.15))
+  (gr_arc (start 139 65.25) (end 139 66.25) (angle -180) (layer Edge.Cuts) (width 0.15))
+  (gr_arc (start 136.5 65.25) (end 136.5 64.25) (angle -180) (layer Edge.Cuts) (width 0.15))
   (gr_text "LED\nDATA54\nDATA36\nDATA12\n3.3V\n5V" (at 128.75 59) (layer F.SilkS)
     (effects (font (size 1.5 1.5) (thickness 0.3)) (justify left))
@@
     (effects (font (size 1.5 1.5) (thickness 0.3)) (justify right))
   )
-  (gr_line (start 90.75 47.5) (end 157.5 47.5) (layer Edge.Cuts) (width 0.15))
-  (gr_line (start 90.75 69.5) (end 90.75 47.5) (layer Edge.Cuts) (width 0.15))
-  (gr_line (start 157.5 69.5) (end 90.75 69.5) (layer Edge.Cuts) (width 0.15))
-  (gr_line (start 157.5 47.5) (end 157.5 69.5) (layer Edge.Cuts) (width 0.15))
+  (gr_line (start 91.75 47.5) (end 141.5 47.5) (layer Edge.Cuts) (width 0.15))
+  (gr_line (start 90.75 68.5) (end 90.75 48.5) (layer Edge.Cuts) (width 0.15))
+  (gr_line (start 141.5 69.5) (end 91.75 69.5) (layer Edge.Cuts) (width 0.15))
+  (gr_line (start 142.5 48.5) (end 142.5 68.5) (layer Edge.Cuts) (width 0.15))
   (via (at 116.5 59.75) (size 0.6) (drill 0.3) (layers F.Cu B.Cu) (net 1))
   (via (at 116.5 58.25) (size 0.6) (drill 0.3) (layers F.Cu B.Cu) (net 1))
@@
   (segment (start 114.095 63.75) (end 114 63.845) (width 0.2) (layer F.Cu) (net 24))
   (segment (start 115.75 63.75) (end 114.095 63.75) (width 0.2) (layer F.Cu) (net 24))
+  (segment (start 112.75 64.25) (end 112.75 67.25) (width 0.2) (layer F.Cu) (net 24))
+  (segment (start 114 63.845) (end 113.155 63.845) (width 0.2) (layer F.Cu) (net 24) (status 1000000))
+  (segment (start 113.155 67.655) (end 114 67.655) (width 0.2) (layer F.Cu) (net 24) (status 1000000))
+  (segment (start 112.75 67.25) (end 113.155 67.655) (width 0.2) (layer F.Cu) (net 24) (status 1000000))
+  (segment (start 113.155 63.845) (end 112.75 64.25) (width 0.2) (layer F.Cu) (net 24))
   (segment (start 114.095 58.25) (end 114 58.345) (width 0.2) (layer F.Cu) (net 25))
   (segment (start 115.75 58.25) (end 114.095 58.25) (width 0.2) (layer F.Cu) (net 25))
@@
   (segment (start 114.095 52.75) (end 114 52.845) (width 0.2) (layer F.Cu) (net 26))
   (segment (start 115.75 52.75) (end 114.095 52.75) (width 0.2) (layer F.Cu) (net 26))
-  (segment (start 112.75 64.25) (end 112.75 67.25) (width 0.2) (layer F.Cu) (net 24))
-  (segment (start 114 63.845) (end 113.155 63.845) (width 0.2) (layer F.Cu) (net 24) (status 1000000))
-  (segment (start 113.155 67.655) (end 114 67.655) (width 0.2) (layer F.Cu) (net 24) (status 1000000))
-  (segment (start 112.75 67.25) (end 113.155 67.655) (width 0.2) (layer F.Cu) (net 24) (status 1000000))
-  (segment (start 113.155 63.845) (end 112.75 64.25) (width 0.2) (layer F.Cu) (net 24))
   (zone (net 1) (net_name GND) (layer F.Cu) (hatch edge 0.508)
     (connect_pads (clearance 0.2))
@@
     (polygon
       (pts
-        (xy 90.75 47.5) (xy 157.5 47.5) (xy 157.5 69.5) (xy 90.75 69.5)
+        (xy 90.75 47.5) (xy 142.5 47.5) (xy 142.5 69.5) (xy 90.75 69.5)
       )
     )
@@
     (polygon
       (pts
-        (xy 90.75 47.5) (xy 157.5 47.5) (xy 157.5 69.5) (xy 90.75 69.5)
+        (xy 90.75 47.5) (xy 142.5 47.5) (xy 142.5 69.5) (xy 90.75 69.5)
       )
     )

Commit message: hw
Parts:
- JP1, JP2, JP3: footprint stmbl:SOLDER_JUMPER_0603 -> stmbl:0603_jumper
Changed lines of the file:
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@@
     (uvia_drill 0.1)
   )
-  (module stmbl:SOLDER_JUMPER_0603 (layer F.Cu)
+  (module stmbl:0603_jumper (layer F.Cu)
     (at 116.5 57)
-    (attr virtual)
-    (fp_text reference JP3 (at 0.244 -1.612) (layer F.SilkS)
+    (descr "Capacitor SMD 0603, reflow soldering, AVX (see smccp.pdf)")
+    (tags "capacitor 0603")
+    (attr smd)
+    (fp_text reference JP3 (at -0.834 1.416) (layer F.SilkS)
       (effects (font (size 0.8 0.8) (thickness 0.2)))
     )
-    (fp_text value Jumper_NO_Small (at 0 -2) (layer F.Fab)
+    (fp_text value Jumper_NO_Small (at 0 1.4) (layer F.Fab)
       (effects (font (size 1 1) (thickness 0.15)))
     )
-    (fp_line (start -0.75 0) (end 0.75 0) (layer F.Mask) (width 0.45))
-    (fp_line (start -0.25 0) (end -0.2 0) (layer F.Cu) (width 0.25))
-    (fp_line (start 0.25 0) (end 0.2 0) (layer F.Cu) (width 0.25))
-    (pad 1 smd roundrect (at -0.75 0) (size 1 0.8) (layers F.Cu F.Paste F.Mask) (roundrect_rratio 0.25)
+    (fp_line (start -1.3 -0.6) (end 1.3 -0.6) (layer F.CrtYd) (width 0.05))
+    (fp_line (start -1.3 0.6) (end 1.3 0.6) (layer F.CrtYd) (width 0.05))
+    (fp_line (start -1.3 -0.6) (end -1.3 0.6) (layer F.CrtYd) (width 0.05))
+    (fp_line (start 1.3 -0.6) (end 1.3 0.6) (layer F.CrtYd) (width 0.05))
+    (pad 2 smd roundrect (at 0.75 0) (size 0.75 0.25) (drill (offset -0.25 0)) (layers F.Cu F.Paste F.Mask) (roundrect_rratio 0.25)
+      (net 3 +5V))
+    (pad 1 smd roundrect (at -0.75 0) (size 0.75 0.25) (drill (offset 0.25 0)) (layers F.Cu F.Paste F.Mask) (roundrect_rratio 0.25)
       (net 23 EN_54))
-    (pad 2 smd roundrect (at 0.75 0) (size 1 0.8) (layers F.Cu F.Paste F.Mask) (roundrect_rratio 0.25)
+    (pad 2 smd roundrect (at 0.75 0) (size 0.59 0.8) (layers F.Cu F.Paste F.Mask) (roundrect_rratio 0.25)
       (net 3 +5V))
+    (pad 1 smd roundrect (at -0.75 0) (size 0.59 0.8) (layers F.Cu F.Paste F.Mask) (roundrect_rratio 0.25)
+      (net 23 EN_54))
   )
-  (module stmbl:SOLDER_JUMPER_0603 (layer F.Cu)
+  (module stmbl:0603_jumper (layer F.Cu)
     (at 116.5 62.5)
-    (attr virtual)
-    (fp_text reference JP2 (at 0.244 -1.612) (layer F.SilkS)
+    (descr "Capacitor SMD 0603, reflow soldering, AVX (see smccp.pdf)")
+    (tags "capacitor 0603")
+    (attr smd)
+    (fp_text reference JP2 (at -0.834 1.416) (layer F.SilkS)
       (effects (font (size 0.8 0.8) (thickness 0.2)))
     )
-    (fp_text value Jumper_NO_Small (at 0 -2) (layer F.Fab)
+    (fp_text value Jumper_NO_Small (at 0 1.4) (layer F.Fab)
       (effects (font (size 1 1) (thickness 0.15)))
     )
-    (fp_line (start -0.75 0) (end 0.75 0) (layer F.Mask) (width 0.45))
-    (fp_line (start -0.25 0) (end -0.2 0) (layer F.Cu) (width 0.25))
-    (fp_line (start 0.25 0) (end 0.2 0) (layer F.Cu) (width 0.25))
-    (pad 1 smd roundrect (at -0.75 0) (size 1 0.8) (layers F.Cu F.Paste F.Mask) (roundrect_rratio 0.25)
+    (fp_line (start -1.3 -0.6) (end 1.3 -0.6) (layer F.CrtYd) (width 0.05))
+    (fp_line (start -1.3 0.6) (end 1.3 0.6) (layer F.CrtYd) (width 0.05))
+    (fp_line (start -1.3 -0.6) (end -1.3 0.6) (layer F.CrtYd) (width 0.05))
+    (fp_line (start 1.3 -0.6) (end 1.3 0.6) (layer F.CrtYd) (width 0.05))
+    (pad 2 smd roundrect (at 0.75 0) (size 0.75 0.25) (drill (offset -0.25 0)) (layers F.Cu F.Paste F.Mask) (roundrect_rratio 0.25)
+      (net 3 +5V))
+    (pad 1 smd roundrect (at -0.75 0) (size 0.75 0.25) (drill (offset 0.25 0)) (layers F.Cu F.Paste F.Mask) (roundrect_rratio 0.25)
       (net 22 EN_36))
-    (pad 2 smd roundrect (at 0.75 0) (size 1 0.8) (layers F.Cu F.Paste F.Mask) (roundrect_rratio 0.25)
+    (pad 2 smd roundrect (at 0.75 0) (size 0.59 0.8) (layers F.Cu F.Paste F.Mask) (roundrect_rratio 0.25)
       (net 3 +5V))
+    (pad 1 smd roundrect (at -0.75 0) (size 0.59 0.8) (layers F.Cu F.Paste F.Mask) (roundrect_rratio 0.25)
+      (net 22 EN_36))
   )
-  (module stmbl:SOLDER_JUMPER_0603 (layer F.Cu)
+  (module stmbl:0603_jumper (layer F.Cu)
     (at 116.5 68)
-    (attr virtual)
-    (fp_text reference JP1 (at 0.244 -1.612) (layer F.SilkS)
+    (descr "Capacitor SMD 0603, reflow soldering, AVX (see smccp.pdf)")
+    (tags "capacitor 0603")
+    (attr smd)
+    (fp_text reference JP1 (at -0.834 1.416) (layer F.SilkS)
       (effects (font (size 0.8 0.8) (thickness 0.2)))
     )
-    (fp_text value Jumper_NO_Small (at 0 -2) (layer F.Fab)
+    (fp_text value Jumper_NO_Small (at 0 1.4) (layer F.Fab)
       (effects (font (size 1 1) (thickness 0.15)))
     )
-    (fp_line (start -0.75 0) (end 0.75 0) (layer F.Mask) (width 0.45))
-    (fp_line (start -0.25 0) (end -0.2 0) (layer F.Cu) (width 0.25))
-    (fp_line (start 0.25 0) (end 0.2 0) (layer F.Cu) (width 0.25))
-    (pad 1 smd roundrect (at -0.75 0) (size 1 0.8) (layers F.Cu F.Paste F.Mask) (roundrect_rratio 0.25)
+    (fp_line (start -1.3 -0.6) (end 1.3 -0.6) (layer F.CrtYd) (width 0.05))
+    (fp_line (start -1.3 0.6) (end 1.3 0.6) (layer F.CrtYd) (width 0.05))
+    (fp_line (start -1.3 -0.6) (end -1.3 0.6) (layer F.CrtYd) (width 0.05))
+    (fp_line (start 1.3 -0.6) (end 1.3 0.6) (layer F.CrtYd) (width 0.05))
+    (pad 2 smd roundrect (at 0.75 0) (size 0.75 0.25) (drill (offset -0.25 0)) (layers F.Cu F.Paste F.Mask) (roundrect_rratio 0.25)
+      (net 3 +5V))
+    (pad 1 smd roundrect (at -0.75 0) (size 0.75 0.25) (drill (offset 0.25 0)) (layers F.Cu F.Paste F.Mask) (roundrect_rratio 0.25)
       (net 21 EN_12))
-    (pad 2 smd roundrect (at 0.75 0) (size 1 0.8) (layers F.Cu F.Paste F.Mask) (roundrect_rratio 0.25)
+    (pad 2 smd roundrect (at 0.75 0) (size 0.59 0.8) (layers F.Cu F.Paste F.Mask) (roundrect_rratio 0.25)
       (net 3 +5V))
+    (pad 1 smd roundrect (at -0.75 0) (size 0.59 0.8) (layers F.Cu F.Paste F.Mask) (roundrect_rratio 0.25)
+      (net 21 EN_12))
   )
   (module stmbl:C_0603 (layer F.Cu)

Commit message: jlc export
Parts:
- renumbered C2 to C401, C3 to C402, C1 to C403, C4 to C404, C5 to C405, C6 to C406, C7 to C407, C8 to C408, C9 to C409, J1 to J401, J2 to J402, JP1 to JP401, JP2 to JP402, JP3 to JP403, R2 to R401, R1 to R402, R3 to R403, R4 to R404, R5 to R405, R6 to R406, R7 to R407, R8 to R408, R9 to R409, R10 to R410, R11 to R411, R12 to R412, R13 to R413, R14 to R414, R15 to R415, U1 to U401, U2 to U402, U3 to U403, U4 to U404
Other:
- board text added: "+/- 1/2 SIN RX or 3/6 COS CK gr 5/4 REF TX bl 7/8 VCC br"
- board text added: "EN12"
- board text added: "EN36"
- board text added: "EN54"
- board text added: "STMBL RS485 BOB V1.0"
