File: rs485/pcb.sch (KiCad schematic (older format))
At the start: 18 parts, among them J1 RJ45_LED, J2 CONN_02X06_Odd_Even, U1 LDO

Commit message: hw
Connections:
- net +3V3: no longer R2.2
- net +5V: now also R2.2
Changed lines of the file:
@@
 	2950 1050 3350 1050
-$Comp
-L stmbl:+3.3V #PWR0102
-U 1 1 5E6DC004
-P 900 2150
-F 0 "#PWR0102" H 900 2000 50  0001 C CNN
-F 1 "+3.3V" V 915 2278 50  0000 L CNN
-F 2 "" H 900 2150 50  0001 C CNN
-F 3 "" H 900 2150 50  0001 C CNN
-	1    900  2150
-	0    -1   -1   0
-$EndComp
 $Comp
 L stmbl:+3.3V #PWR0103
@@
 Wire Wire Line
 	6450 2650 6550 2650
+$Comp
+L stmbl:+5V #PWR?
+U 1 1 5E987A68
+P 900 2150
+F 0 "#PWR?" H 900 2000 50  0001 C CNN
+F 1 "+5V" H 915 2323 50  0000 C CNN
+F 2 "" H 900 2150 50  0001 C CNN
+F 3 "" H 900 2150 50  0001 C CNN
+	1    900  2150
+	0    -1   -1   0
+$EndComp
 $EndSCHEMATC

Commit message: parts
Parts:
- C1, C3, C4, C5: LCSC (none) -> C14663
- C2, C6: LCSC (none) -> C15850
- R1, R2: LCSC (none) -> C23204
- R3, R4, R5, R6, R7, R8, R9: LCSC (none) -> C22787
- U1: LCSC (none) -> C9055
Changed lines of the file:
@@
 F 2 "stmbl:C_0603" H 2165 3459 50  0001 L CNN
 F 3 "" H 2050 3550 50  0001 C CNN
+F 4 "C14663" H 2050 3550 50  0001 C CNN "LCSC"
 	1    2050 3550
 	1    0    0    -1
@@
 F 2 "stmbl:C_0603" V 1680 3550 50  0001 C CNN
 F 3 "" H 1750 3550 50  0001 C CNN
+F 4 "C22787" H 1750 3550 50  0001 C CNN "LCSC"
 	1    1750 3550
 	1    0    0    -1
@@
 F 2 "stmbl:C_0603" V 1080 2850 50  0001 C CNN
 F 3 "" H 1150 2850 50  0001 C CNN
+F 4 "C23204" H 1150 2850 50  0001 C CNN "LCSC"
 	1    1150 2850
 	0    1    1    0
@@
 F 2 "stmbl:C_0603" V 1080 2150 50  0001 C CNN
 F 3 "" H 1150 2150 50  0001 C CNN
+F 4 "C23204" H 1150 2150 50  0001 C CNN "LCSC"
 	1    1150 2150
 	0    1    1    0
@@
 F 2 "stmbl:C_0805" H 838 1150 50  0001 C CNN
 F 3 "" H 800 1300 50  0001 C CNN
+F 4 "C15850" H 800 1300 50  0001 C CNN "LCSC"
 	1    800  1300
 	1    0    0    -1
@@
 F 2 "stmbl:SOT-23-5" H 2550 900 50  0001 C CIN
 F 3 "" H 1900 1150 50  0000 C CNN
+F 4 "C9055" H 1900 1150 50  0001 C CNN "LCSC"
 	1    1900 1150
 	1    0    0    -1
@@
 F 2 "stmbl:C_0603" H 2615 1159 50  0001 L CNN
 F 3 "" H 2500 1250 50  0001 C CNN
+F 4 "C14663" H 2500 1250 50  0001 C CNN "LCSC"
 	1    2500 1250
 	0    -1   -1   0
@@
 F 2 "stmbl:C_0603" H 3065 1209 50  0001 L CNN
 F 3 "" H 2950 1300 50  0001 C CNN
+F 4 "C14663" H 2950 1300 50  0001 C CNN "LCSC"
 	1    2950 1300
 	1    0    0    -1
@@
 F 2 "stmbl:C_0805" H 3388 1150 50  0001 C CNN
 F 3 "" H 3350 1300 50  0001 C CNN
+F 4 "C15850" H 3350 1300 50  0001 C CNN "LCSC"
 	1    3350 1300
 	1    0    0    -1
@@
 F 2 "stmbl:C_0603" H 1315 1209 50  0001 L CNN
 F 3 "" H 1200 1300 50  0001 C CNN
+F 4 "C14663" H 1200 1300 50  0001 C CNN "LCSC"
 	1    1200 1300
 	1    0    0    -1
@@
 F 2 "stmbl:C_0603" V 5230 2450 50  0001 C CNN
 F 3 "" H 5300 2450 50  0001 C CNN
+F 4 "C22787" H 5300 2450 50  0001 C CNN "LCSC"
 	1    5300 2450
 	0    1    1    0
@@
 F 2 "stmbl:C_0603" V 5230 2550 50  0001 C CNN
 F 3 "" H 5300 2550 50  0001 C CNN
+F 4 "C22787" H 5300 2550 50  0001 C CNN "LCSC"
 	1    5300 2550
 	0    1    1    0
@@
 F 2 "stmbl:C_0603" V 5230 2650 50  0001 C CNN
 F 3 "" H 5300 2650 50  0001 C CNN
+F 4 "C22787" H 5300 2650 50  0001 C CNN "LCSC"
 	1    5300 2650
 	0    1    1    0
@@
 F 2 "stmbl:C_0603" V 6230 2450 50  0001 C CNN
 F 3 "" H 6300 2450 50  0001 C CNN
+F 4 "C22787" H 6300 2450 50  0001 C CNN "LCSC"
 	1    6300 2450
 	0    1    1    0
@@
 F 2 "stmbl:C_0603" V 6230 2550 50  0001 C CNN
 F 3 "" H 6300 2550 50  0001 C CNN
+F 4 "C22787" H 6300 2550 50  0001 C CNN "LCSC"
 	1    6300 2550
 	0    1    1    0
@@
 F 2 "stmbl:C_0603" V 6230 2650 50  0001 C CNN
 F 3 "" H 6300 2650 50  0001 C CNN
+F 4 "C22787" H 6300 2650 50  0001 C CNN "LCSC"
 	1    6300 2650
 	0    1    1    0

Commit message: jlc export
Parts:
- renumbered C2 to C401, C3 to C402, C1 to C403, C4 to C404, C5 to C405, C6 to C406, J1 to J401, J2 to J402, R2 to R401, R1 to R402, R3 to R403, R4 to R404, R5 to R405, R6 to R406, R7 to R407, R8 to R408, R9 to R409, U1 to U401
Changed lines of the file:
@@
 $EndDescr
 $Comp
-L stmbl:RJ45_LED J1
+L stmbl:RJ45_LED J401
 U 1 1 5E3EE2C2
 P 1900 2550
-F 0 "J1" V 1275 2550 50  0000 C CNN
+F 0 "J401" V 1275 2550 50  0000 C CNN
 F 1 "RJ45_LED" V 1366 2550 50  0000 C CNN
 F 2 "stmbl:RJ45_LED" V 1359 2550 60  0001 C CNN
@@
 6
 $Comp
-L stmbl:GND #PWR07
+L stmbl:GND #PWR0409
 U 1 1 5E49521C
 P 2500 2950
-F 0 "#PWR07" H 2500 2700 50  0001 C CNN
+F 0 "#PWR0409" H 2500 2700 50  0001 C CNN
 F 1 "GND" V 2505 2822 50  0000 R CNN
 F 2 "" H 2500 2950 50  0001 C CNN
@@
 $EndComp
 $Comp
-L stmbl:+5V #PWR06
+L stmbl:+5V #PWR0408
 U 1 1 5E495775
 P 2500 2850
-F 0 "#PWR06" H 2500 2700 50  0001 C CNN
+F 0 "#PWR0408" H 2500 2700 50  0001 C CNN
 F 1 "+5V" V 2515 2978 50  0000 L CNN
 F 2 "" H 2500 2850 50  0001 C CNN
@@
 $EndComp
 $Comp
-L stmbl:GND #PWR05
+L stmbl:GND #PWR0407
 U 1 1 5E4B51FF
 P 1900 3950
-F 0 "#PWR05" H 1900 3700 50  0001 C CNN
+F 0 "#PWR0407" H 1900 3700 50  0001 C CNN
 F 1 "GND" H 1905 3777 50  0000 C CNN
 F 2 "" H 1900 3950 50  0001 C CNN
@@
 $EndComp
 $Comp
-L stmbl:C C1
+L stmbl:C C403
 U 1 1 5E4B57A3
 P 2050 3550
-F 0 "C1" H 2165 3596 50  0000 L CNN
+F 0 "C403" H 2165 3596 50  0000 L CNN
 F 1 "100n" H 2165 3505 50  0000 L CNN
 F 2 "stmbl:C_0603" H 2165 3459 50  0001 L CNN
@@
 $EndComp
 $Comp
-L stmbl:R R3
+L stmbl:R R403
 U 1 1 5E4B74DA
 P 1750 3550
-F 0 "R3" H 1820 3596 50  0000 L CNN
+F 0 "R403" H 1820 3596 50  0000 L CNN
 F 1 "120" H 1820 3505 50  0000 L CNN
 F 2 "stmbl:C_0603" V 1680 3550 50  0001 C CNN
@@
 Connection ~ 1750 3300
 $Comp
-L stmbl:GND #PWR03
+L stmbl:GND #PWR0405
 U 1 1 5E5475A7
 P 1300 2950
-F 0 "#PWR03" H 1300 2700 50  0001 C CNN
+F 0 "#PWR0405" H 1300 2700 50  0001 C CNN
 F 1 "GND" V 1305 2822 50  0000 R CNN
 F 2 "" H 1300 2950 50  0001 C CNN
@@
 $EndComp
 $Comp
-L stmbl:GND #PWR02
+L stmbl:GND #PWR0404
 U 1 1 5E547A90
 P 1300 2250
-F 0 "#PWR02" H 1300 2000 50  0001 C CNN
+F 0 "#PWR0404" H 1300 2000 50  0001 C CNN
 F 1 "GND" V 1305 2122 50  0000 R CNN
 F 2 "" H 1300 2250 50  0001 C CNN
@@
 	1300 2850 1400 2850
 $Comp
-L stmbl:R R1
+L stmbl:R R402
 U 1 1 5E565B57
 P 1150 2850
-F 0 "R1" V 1050 2850 50  0000 C CNN
+F 0 "R402" V 1050 2850 50  0000 C CNN
 F 1 "560" V 1150 2850 50  0000 C CNN
 F 2 "stmbl:C_0603" V 1080 2850 50  0001 C CNN
@@
 	900  2850 1000 2850
 $Comp
-L stmbl:R R2
+L stmbl:R R401
 U 1 1 5E56E034
 P 1150 2150
-F 0 "R2" V 1050 2150 50  0000 C CNN
+F 0 "R401" V 1050 2150 50  0000 C CNN
 F 1 "560" V 1150 2150 50  0000 C CNN
 F 2 "stmbl:C_0603" V 1080 2150 50  0001 C CNN
@@
 	2400 2950 2500 2950
 $Comp
-L stmbl:C C2
+L stmbl:C C401
 U 1 1 5E6C67E4
 P 800 1300
-F 0 "C2" H 915 1346 50  0000 L CNN
+F 0 "C401" H 915 1346 50  0000 L CNN
 F 1 "10u" H 915 1255 50  0000 L CNN
 F 2 "stmbl:C_0805" H 838 1150 50  0001 C CNN
@@
 $EndComp
 $Comp
-L stmbl:+5V #PWR0101
+L stmbl:+5V #PWR0401
 U 1 1 5E6C71AF
 P 800 950
-F 0 "#PWR0101" H 800 800 50  0001 C CNN
+F 0 "#PWR0401" H 800 800 50  0001 C CNN
 F 1 "+5V" H 815 1123 50  0000 C CNN
 F 2 "" H 800 950 50  0001 C CNN
@@
 	800  1550 800  1650
 $Comp
-L stmbl:LDO U1
+L stmbl:LDO U401
 U 1 1 5E6CADAF
 P 1900 1150
-F 0 "U1" H 1900 1475 50  0000 C CNN
+F 0 "U401" H 1900 1475 50  0000 C CNN
 F 1 "LDO" H 1900 1384 50  0000 C CNN
 F 2 "stmbl:SOT-23-5" H 2550 900 50  0001 C CIN
@@
 $EndComp
 $Comp
-L stmbl:C C4
+L stmbl:C C404
 U 1 1 5E6CE826
 P 2500 1250
-F 0 "C4" V 2752 1250 50  0000 C CNN
+F 0 "C404" V 2752 1250 50  0000 C CNN
 F 1 "100n" V 2661 1250 50  0000 C CNN
 F 2 "stmbl:C_0603" H 2615 1159 50  0001 L CNN
@@
 $EndComp
 $Comp
-L stmbl:C C5
+L stmbl:C C405
 U 1 1 5E6CEEA4
 P 2950 1300
-F 0 "C5" V 3202 1300 50  0000 C CNN
+F 0 "C405" V 3202 1300 50  0000 C CNN
 F 1 "100n" V 3111 1300 50  0000 C CNN
 F 2 "stmbl:C_0603" H 3065 1209 50  0001 L CNN
@@
 $EndComp
 $Comp
-L stmbl:C C6
+L stmbl:C C406
 U 1 1 5E6CFBBB
 P 3350 1300
-F 0 "C6" H 3465 1346 50  0000 L CNN
+F 0 "C406" H 3465 1346 50  0000 L CNN
 F 1 "10u" H 3465 1255 50  0000 L CNN
 F 2 "stmbl:C_0805" H 3388 1150 50  0001 C CNN
@@
 	2950 1050 3350 1050
 $Comp
-L stmbl:+3.3V #PWR0103
+L stmbl:+3.3V #PWR0410
 U 1 1 5E6DC800
 P 3350 950
-F 0 "#PWR0103" H 3350 800 50  0001 C CNN
+F 0 "#PWR0410" H 3350 800 50  0001 C CNN
 F 1 "+3.3V" H 3365 1123 50  0000 C CNN
 F 2 "" H 3350 950 50  0001 C CNN
@@
 Connection ~ 3350 1050
 $Comp
-L stmbl:C C3
+L stmbl:C C402
 U 1 1 5E6E1141
 P 1200 1300
-F 0 "C3" V 1452 1300 50  0000 C CNN
+F 0 "C402" V 1452 1300 50  0000 C CNN
 F 1 "100n" V 1361 1300 50  0000 C CNN
 F 2 "stmbl:C_0603" H 1315 1209 50  0001 L CNN
@@
 $EndSheet
 $Comp
-L stmbl:GND #PWR0104
+L stmbl:GND #PWR0402
 U 1 1 5E707AB7
 P 800 1650
-F 0 "#PWR0104" H 800 1400 50  0001 C CNN
+F 0 "#PWR0402" H 800 1400 50  0001 C CNN
 F 1 "GND" H 805 1477 50  0000 C CNN
 F 2 "" H 800 1650 50  0001 C CNN
@@
 	1650 3300 1750 3300
 $Comp
-L stmbl:GNDS #PWR04
+L stmbl:GNDS #PWR0406
 U 1 1 5E4CAF52
 P 1650 3300
-F 0 "#PWR04" H 1650 3050 50  0001 C CNN
+F 0 "#PWR0406" H 1650 3050 50  0001 C CNN
 F 1 "GNDS" V 1655 3172 50  0000 R CNN
 F 2 "" H 1650 3300 50  0001 C CNN
@@
 5
 $Comp
-L stmbl:+5V #PWR0105
+L stmbl:+5V #PWR0411
 U 1 1 5E718308
 P 5450 2250
-F 0 "#PWR0105" H 5450 2100 50  0001 C CNN
+F 0 "#PWR0411" H 5450 2100 50  0001 C CNN
 F 1 "+5V" H 5465 2423 50  0000 C CNN
 F 2 "" H 5450 2250 50  0001 C CNN
@@
 $EndComp
 $Comp
-L stmbl:+3.3V #PWR0106
+L stmbl:+3.3V #PWR0412
 U 1 1 5E718B54
 P 5450 2350
-F 0 "#PWR0106" H 5450 2200 50  0001 C CNN
+F 0 "#PWR0412" H 5450 2200 50  0001 C CNN
 F 1 "+3.3V" V 5465 2478 50  0000 L CNN
 F 2 "" H 5450 2350 50  0001 C CNN
@@
 $EndComp
 $Comp
-L stmbl:GND #PWR0107
+L stmbl:GND #PWR0413
 U 1 1 5E71942F
 P 6150 2250
-F 0 "#PWR0107" H 6150 2000 50  0001 C CNN
+F 0 "#PWR0413" H 6150 2000 50  0001 C CNN
 F 1 "GND" V 6155 2122 50  0000 R CNN
 F 2 "" H 6150 2250 50  0001 C CNN
@@
 $EndComp
 $Comp
-L stmbl:GNDS #PWR0108
+L stmbl:GNDS #PWR0415
 U 1 1 5E71AEC4
 P 6150 2750
-F 0 "#PWR0108" H 6150 2500 50  0001 C CNN
+F 0 "#PWR0415" H 6150 2500 50  0001 C CNN
 F 1 "GNDS" V 6155 2622 50  0000 R CNN
 F 2 "" H 6150 2750 50  0001 C CNN
@@
 EN_54
 $Comp
-L stmbl:CONN_02X06_Odd_Even J2
+L stmbl:CONN_02X06_Odd_Even J402
 U 1 1 5E71C335
 P 5750 2450
-F 0 "J2" H 5800 2867 50  0000 C CNN
+F 0 "J402" H 5800 2867 50  0000 C CNN
 F 1 "CONN_02X06_Odd_Even" H 5800 2776 50  0000 C CNN
 F 2 "stmbl:Pin_Header_RM2.54_2x6_UP" H 5750 2450 50  0001 C CNN
@@
 $EndComp
 $Comp
-L stmbl:GND #PWR0109
+L stmbl:GND #PWR0414
 U 1 1 5E71D8B4
 P 6150 2350
-F 0 "#PWR0109" H 6150 2100 50  0001 C CNN
+F 0 "#PWR0414" H 6150 2100 50  0001 C CNN
 F 1 "GND" V 6155 2222 50  0000 R CNN
 F 2 "" H 6150 2350 50  0001 C CNN
@@
 	6050 2250 6150 2250
 $Comp
-L stmbl:R R4
+L stmbl:R R404
 U 1 1 5E731B0B
 P 5300 2450
-F 0 "R4" V 5250 2550 50  0000 L CNN
+F 0 "R404" V 5250 2550 50  0000 L CNN
 F 1 "120" V 5300 2400 50  0000 L CNN
 F 2 "stmbl:C_0603" V 5230 2450 50  0001 C CNN
@@
 $EndComp
 $Comp
-L stmbl:R R5
+L stmbl:R R405
 U 1 1 5E73BE2C
 P 5300 2550
-F 0 "R5" V 5250 2650 50  0000 L CNN
+F 0 "R405" V 5250 2650 50  0000 L CNN
 F 1 "120" V 5300 2500 50  0000 L CNN
 F 2 "stmbl:C_0603" V 5230 2550 50  0001 C CNN
@@
 $EndComp
 $Comp
-L stmbl:R R6
+L stmbl:R R406
 U 1 1 5E73C150
 P 5300 2650
-F 0 "R6" V 5250 2750 50  0000 L CNN
+F 0 "R406" V 5250 2750 50  0000 L CNN
 F 1 "120" V 5300 2600 50  0000 L CNN
 F 2 "stmbl:C_0603" V 5230 2650 50  0001 C CNN
@@
 	5050 2450 5150 2450
 $Comp
-L stmbl:R R7
+L stmbl:R R407
 U 1 1 5E7442F2
 P 6300 2450
-F 0 "R7" V 6250 2550 50  0000 L CNN
+F 0 "R407" V 6250 2550 50  0000 L CNN
 F 1 "120" V 6300 2400 50  0000 L CNN
 F 2 "stmbl:C_0603" V 6230 2450 50  0001 C CNN
@@
 $EndComp
 $Comp
-L stmbl:R R8
+L stmbl:R R408
 U 1 1 5E7442F8
 P 6300 2550
-F 0 "R8" V 6250 2650 50  0000 L CNN
+F 0 "R408" V 6250 2650 50  0000 L CNN
 F 1 "120" V 6300 2500 50  0000 L CNN
 F 2 "stmbl:C_0603" V 6230 2550 50  0001 C CNN
@@
 $EndComp
 $Comp
-L stmbl:R R9
+L stmbl:R R409
 U 1 1 5E7442FE
 P 6300 2650
-F 0 "R9" V 6250 2750 50  0000 L CNN
+F 0 "R409" V 6250 2750 50  0000 L CNN
 F 1 "120" V 6300 2600 50  0000 L CNN
 F 2 "stmbl:C_0603" V 6230 2650 50  0001 C CNN
@@
 	6450 2650 6550 2650
 $Comp
-L stmbl:+5V #PWR?
+L stmbl:+5V #PWR0403
 U 1 1 5E987A68
 P 900 2150
-F 0 "#PWR?" H 900 2000 50  0001 C CNN
+F 0 "#PWR0403" H 900 2000 50  0001 C CNN
 F 1 "+5V" H 915 2323 50  0000 C CNN
 F 2 "" H 900 2150 50  0001 C CNN
