File: rs485/rs485.sch (KiCad schematic (older format))
At the start: 5 parts, among them U2 sp485

Commit message: parts
Parts:
- C7: LCSC (none) -> C14663
- R10: LCSC (none) -> C22787
- R11: LCSC (none) -> C21190
- U2: LCSC (none) -> C6855
Changed lines of the file:
@@
 F 2 "stmbl:C_0603" H 5815 3459 50  0001 L CNN
 F 3 "" H 5700 3550 50  0001 C CNN
+F 4 "C14663" H 5700 3550 50  0001 C CNN "LCSC"
 	1    5700 3550
 	0    -1   -1   0
@@
 F 2 "stmbl:SOIC-8-N" H 5700 4333 50  0001 C CIN
 F 3 "" H 5700 4050 50  0001 C CNN
+F 4 "C6855" H 5700 4050 50  0001 C CNN "LCSC"
 	1    5700 4050
 	-1   0    0    -1
@@
 F 2 "stmbl:C_0603" V 4780 4050 50  0001 C CNN
 F 3 "" H 4850 4050 50  0001 C CNN
+F 4 "C22787" H 4850 4050 50  0001 C CNN "LCSC"
 	1    4850 4050
 	1    0    0    -1
@@
 F 2 "stmbl:R_0603" V 6780 3550 50  0001 C CNN
 F 3 "" H 6850 3550 50  0001 C CNN
+F 4 "C21190" H 6850 3550 50  0001 C CNN "LCSC"
 	1    6850 3550
 	0    1    1    0

Commit message: hw
Parts:
- JP1: footprint stmbl:SOLDER_JUMPER_0603 -> stmbl:0603_jumper
Changed lines of the file:
@@
 F 0 "JP1" H 6800 3550 50  0000 C CNN
 F 1 "Jumper_NO_Small" H 6810 3590 50  0001 C CNN
-F 2 "stmbl:SOLDER_JUMPER_0603" H 6800 3650 50  0001 C CNN
+F 2 "stmbl:0603_jumper" H 6800 3650 50  0001 C CNN
 F 3 "" H 6800 3650 50  0000 C CNN
 	1    6800 3650

Commit message: jlc export
Parts:
- renumbered C7 to C407, JP1 to JP401, R10 to R410, R11 to R411, U2 to U402
Changed lines of the file:
@@
 P 5700 3550
 AR Path="/5E703907" Ref="C?"  Part="1"
-AR Path="/5E701549/5E703907" Ref="C7"  Part="1"
-AR Path="/5E7141F1/5E703907" Ref="C8"  Part="1"
-AR Path="/5E715706/5E703907" Ref="C9"  Part="1"
-F 0 "C7" V 5952 3550 50  0000 C CNN
+AR Path="/5E701549/5E703907" Ref="C407"  Part="1"
+AR Path="/5E7141F1/5E703907" Ref="C408"  Part="1"
+AR Path="/5E715706/5E703907" Ref="C409"  Part="1"
+F 0 "C409" V 5952 3550 50  0000 C CNN
 F 1 "100n" V 5861 3550 50  0000 C CNN
 F 2 "stmbl:C_0603" H 5815 3459 50  0001 L CNN
@@
 $EndComp
 $Comp
-L stmbl:RS485 U2
+L stmbl:RS485 U402
 U 1 1 5E70390D
 P 5700 4050
-AR Path="/5E701549/5E70390D" Ref="U2"  Part="1"
-AR Path="/5E7141F1/5E70390D" Ref="U3"  Part="1"
-AR Path="/5E715706/5E70390D" Ref="U4"  Part="1"
-F 0 "U2" H 5700 4425 50  0000 C CNN
+AR Path="/5E701549/5E70390D" Ref="U402"  Part="1"
+AR Path="/5E7141F1/5E70390D" Ref="U403"  Part="1"
+AR Path="/5E715706/5E70390D" Ref="U404"  Part="1"
+F 0 "U404" H 5700 4425 50  0000 C CNN
 F 1 "sp485" H 5700 4334 50  0000 C CNN
 F 2 "stmbl:SOIC-8-N" H 5700 4333 50  0001 C CIN
@@
 P 5250 3900
 AR Path="/5E703913" Ref="#PWR?"  Part="1"
-AR Path="/5E701549/5E703913" Ref="#PWR0110"  Part="1"
-AR Path="/5E7141F1/5E703913" Ref="#PWR0116"  Part="1"
-AR Path="/5E715706/5E703913" Ref="#PWR0122"  Part="1"
-F 0 "#PWR0110" H 5250 3750 50  0001 C CNN
+AR Path="/5E701549/5E703913" Ref="#PWR0416"  Part="1"
+AR Path="/5E7141F1/5E703913" Ref="#PWR0422"  Part="1"
+AR Path="/5E715706/5E703913" Ref="#PWR0428"  Part="1"
+F 0 "#PWR0428" H 5250 3750 50  0001 C CNN
 F 1 "+5V" V 5265 4028 50  0000 L CNN
 F 2 "" H 5250 3900 50  0001 C CNN
@@
 $EndComp
 $Comp
-L stmbl:GND #PWR0111
+L stmbl:GND #PWR0417
 U 1 1 5E703919
 P 5250 4200
-AR Path="/5E701549/5E703919" Ref="#PWR0111"  Part="1"
-AR Path="/5E7141F1/5E703919" Ref="#PWR0117"  Part="1"
-AR Path="/5E715706/5E703919" Ref="#PWR0123"  Part="1"
-F 0 "#PWR0111" H 5250 3950 50  0001 C CNN
+AR Path="/5E701549/5E703919" Ref="#PWR0417"  Part="1"
+AR Path="/5E7141F1/5E703919" Ref="#PWR0423"  Part="1"
+AR Path="/5E715706/5E703919" Ref="#PWR0429"  Part="1"
+F 0 "#PWR0429" H 5250 3950 50  0001 C CNN
 F 1 "GND" V 5255 4072 50  0000 R CNN
 F 2 "" H 5250 4200 50  0001 C CNN
@@
 P 5950 3550
 AR Path="/5E70392A" Ref="#PWR?"  Part="1"
-AR Path="/5E701549/5E70392A" Ref="#PWR0112"  Part="1"
-AR Path="/5E7141F1/5E70392A" Ref="#PWR0118"  Part="1"
-AR Path="/5E715706/5E70392A" Ref="#PWR0124"  Part="1"
-F 0 "#PWR0112" H 5950 3300 50  0001 C CNN
+AR Path="/5E701549/5E70392A" Ref="#PWR0419"  Part="1"
+AR Path="/5E7141F1/5E70392A" Ref="#PWR0425"  Part="1"
+AR Path="/5E715706/5E70392A" Ref="#PWR0431"  Part="1"
+F 0 "#PWR0431" H 5950 3300 50  0001 C CNN
 F 1 "GND" H 5955 3377 50  0000 C CNN
 F 2 "" H 5950 3550 50  0001 C CNN
@@
 P 5450 3550
 AR Path="/5E703930" Ref="#PWR?"  Part="1"
-AR Path="/5E701549/5E703930" Ref="#PWR0113"  Part="1"
-AR Path="/5E7141F1/5E703930" Ref="#PWR0119"  Part="1"
-AR Path="/5E715706/5E703930" Ref="#PWR0125"  Part="1"
-F 0 "#PWR0113" H 5450 3400 50  0001 C CNN
+AR Path="/5E701549/5E703930" Ref="#PWR0418"  Part="1"
+AR Path="/5E7141F1/5E703930" Ref="#PWR0424"  Part="1"
+AR Path="/5E715706/5E703930" Ref="#PWR0430"  Part="1"
+F 0 "#PWR0430" H 5450 3400 50  0001 C CNN
 F 1 "+5V" H 5465 3723 50  0000 C CNN
 F 2 "" H 5450 3550 50  0001 C CNN
@@
 P 7000 3650
 AR Path="/5E703938" Ref="#PWR?"  Part="1"
-AR Path="/5E701549/5E703938" Ref="#PWR0114"  Part="1"
-AR Path="/5E7141F1/5E703938" Ref="#PWR0120"  Part="1"
-AR Path="/5E715706/5E703938" Ref="#PWR0126"  Part="1"
-F 0 "#PWR0114" H 7000 3500 50  0001 C CNN
+AR Path="/5E701549/5E703938" Ref="#PWR0420"  Part="1"
+AR Path="/5E7141F1/5E703938" Ref="#PWR0426"  Part="1"
+AR Path="/5E715706/5E703938" Ref="#PWR0432"  Part="1"
+F 0 "#PWR0432" H 7000 3500 50  0001 C CNN
 F 1 "+5V" V 7015 3778 50  0000 L CNN
 F 2 "" H 7000 3650 50  0001 C CNN
@@
 P 4850 4050
 AR Path="/5E70393F" Ref="R?"  Part="1"
-AR Path="/5E701549/5E70393F" Ref="R10"  Part="1"
-AR Path="/5E7141F1/5E70393F" Ref="R12"  Part="1"
-AR Path="/5E715706/5E70393F" Ref="R14"  Part="1"
-F 0 "R10" H 4920 4096 50  0000 L CNN
+AR Path="/5E701549/5E70393F" Ref="R410"  Part="1"
+AR Path="/5E7141F1/5E70393F" Ref="R412"  Part="1"
+AR Path="/5E715706/5E70393F" Ref="R414"  Part="1"
+F 0 "R414" H 4920 4096 50  0000 L CNN
 F 1 "120" H 4920 4005 50  0000 L CNN
 F 2 "stmbl:C_0603" V 4780 4050 50  0001 C CNN
@@
 P 6800 3650
 AR Path="/5E703949" Ref="JP?"  Part="1"
-AR Path="/5E701549/5E703949" Ref="JP1"  Part="1"
-AR Path="/5E7141F1/5E703949" Ref="JP2"  Part="1"
-AR Path="/5E715706/5E703949" Ref="JP3"  Part="1"
-F 0 "JP1" H 6800 3550 50  0000 C CNN
+AR Path="/5E701549/5E703949" Ref="JP401"  Part="1"
+AR Path="/5E7141F1/5E703949" Ref="JP402"  Part="1"
+AR Path="/5E715706/5E703949" Ref="JP403"  Part="1"
+F 0 "JP403" H 6800 3550 50  0000 C CNN
 F 1 "Jumper_NO_Small" H 6810 3590 50  0001 C CNN
 F 2 "stmbl:0603_jumper" H 6800 3650 50  0001 C CNN
@@
 P 7100 3550
 AR Path="/5E703950" Ref="#PWR?"  Part="1"
-AR Path="/5E701549/5E703950" Ref="#PWR0115"  Part="1"
-AR Path="/5E7141F1/5E703950" Ref="#PWR0121"  Part="1"
-AR Path="/5E715706/5E703950" Ref="#PWR0127"  Part="1"
-F 0 "#PWR0115" H 7100 3300 50  0001 C CNN
+AR Path="/5E701549/5E703950" Ref="#PWR0421"  Part="1"
+AR Path="/5E7141F1/5E703950" Ref="#PWR0427"  Part="1"
+AR Path="/5E715706/5E703950" Ref="#PWR0433"  Part="1"
+F 0 "#PWR0433" H 7100 3300 50  0001 C CNN
 F 1 "GND" H 7105 3377 50  0000 C CNN
 F 2 "" H 7100 3550 50  0001 C CNN
@@
 P 6850 3550
 AR Path="/5E703959" Ref="R?"  Part="1"
-AR Path="/5E701549/5E703959" Ref="R11"  Part="1"
-AR Path="/5E7141F1/5E703959" Ref="R13"  Part="1"
-AR Path="/5E715706/5E703959" Ref="R15"  Part="1"
-F 0 "R11" V 6750 3550 50  0000 C CNN
+AR Path="/5E701549/5E703959" Ref="R411"  Part="1"
+AR Path="/5E7141F1/5E703959" Ref="R413"  Part="1"
+AR Path="/5E715706/5E703959" Ref="R415"  Part="1"
+F 0 "R415" V 6750 3550 50  0000 C CNN
 F 1 "1k" V 6850 3550 50  0000 C CNN
 F 2 "stmbl:R_0603" V 6780 3550 50  0001 C CNN
